File: pcb/11bitcount.kicad_sch (KiCad schematic)
At the start: 3 parts, among them U15 74HC161, U16 74HC161, U17 74HC161

Commit message: WIP schematic
Parts:
- renumbered U15 to U16, U16 to U17, U17 to U18
Changed lines of the file:
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@@
 		(dnp no)
 		(fields_autoplaced yes)
-		(property "Reference" "#PWR070"
+		(property "Reference" "#PWR085"
 			(at 83.82 77.47 0)
 			(effects
@@
 			(project ""
 				(path "/e63e39d7-6ac0-4ffd-8aa3-1841a4541b55/90e1f016-3c60-4383-aa8d-def9977ac47b/78a99c0a-f468-453e-aea1-d254ed568110"
-					(reference "#PWR070")
-					(unit 1)
-				)
-				(path "/e63e39d7-6ac0-4ffd-8aa3-1841a4541b55/90e1f016-3c60-4383-aa8d-def9977ac47b/d909784a-ae31-4c8f-b386-03ea0f044fee"
-					(reference "#PWR079")
+					(reference "#PWR085")
+					(unit 1)
+				)
+				(path "/e63e39d7-6ac0-4ffd-8aa3-1841a4541b55/90e1f016-3c60-4383-aa8d-def9977ac47b/d909784a-ae31-4c8f-b386-03ea0f044fee"
+					(reference "#PWR094")
 					(unit 1)
 				)
@@
 		(on_board yes)
 		(dnp no)
-		(property "Reference" "#PWR068"
+		(property "Reference" "#PWR083"
 			(at 58.42 43.18 0)
 			(effects
@@
 			(project ""
 				(path "/e63e39d7-6ac0-4ffd-8aa3-1841a4541b55/90e1f016-3c60-4383-aa8d-def9977ac47b/78a99c0a-f468-453e-aea1-d254ed568110"
-					(reference "#PWR068")
-					(unit 1)
-				)
-				(path "/e63e39d7-6ac0-4ffd-8aa3-1841a4541b55/90e1f016-3c60-4383-aa8d-def9977ac47b/d909784a-ae31-4c8f-b386-03ea0f044fee"
-					(reference "#PWR077")
+					(reference "#PWR083")
+					(unit 1)
+				)
+				(path "/e63e39d7-6ac0-4ffd-8aa3-1841a4541b55/90e1f016-3c60-4383-aa8d-def9977ac47b/d909784a-ae31-4c8f-b386-03ea0f044fee"
+					(reference "#PWR092")
 					(unit 1)
 				)
@@
 		(on_board yes)
 		(dnp no)
-		(property "Reference" "U17"
+		(property "Reference" "U18"
 			(at 142.748 76.708 90)
 			(effects
@@
 			(project ""
 				(path "/e63e39d7-6ac0-4ffd-8aa3-1841a4541b55/90e1f016-3c60-4383-aa8d-def9977ac47b/78a99c0a-f468-453e-aea1-d254ed568110"
-					(reference "U17")
-					(unit 1)
-				)
-				(path "/e63e39d7-6ac0-4ffd-8aa3-1841a4541b55/90e1f016-3c60-4383-aa8d-def9977ac47b/d909784a-ae31-4c8f-b386-03ea0f044fee"
-					(reference "U20")
+					(reference "U18")
+					(unit 1)
+				)
+				(path "/e63e39d7-6ac0-4ffd-8aa3-1841a4541b55/90e1f016-3c60-4383-aa8d-def9977ac47b/d909784a-ae31-4c8f-b386-03ea0f044fee"
+					(reference "U21")
 					(unit 1)
 				)
@@
 		(dnp no)
 		(fields_autoplaced yes)
-		(property "Reference" "#PWR073"
+		(property "Reference" "#PWR088"
 			(at 134.62 77.47 0)
 			(effects
@@
 			(project ""
 				(path "/e63e39d7-6ac0-4ffd-8aa3-1841a4541b55/90e1f016-3c60-4383-aa8d-def9977ac47b/78a99c0a-f468-453e-aea1-d254ed568110"
-					(reference "#PWR073")
-					(unit 1)
-				)
-				(path "/e63e39d7-6ac0-4ffd-8aa3-1841a4541b55/90e1f016-3c60-4383-aa8d-def9977ac47b/d909784a-ae31-4c8f-b386-03ea0f044fee"
-					(reference "#PWR082")
+					(reference "#PWR088")
+					(unit 1)
+				)
+				(path "/e63e39d7-6ac0-4ffd-8aa3-1841a4541b55/90e1f016-3c60-4383-aa8d-def9977ac47b/d909784a-ae31-4c8f-b386-03ea0f044fee"
+					(reference "#PWR097")
 					(unit 1)
 				)
@@
 		(on_board yes)
 		(dnp no)
-		(property "Reference" "#PWR069"
+		(property "Reference" "#PWR084"
 			(at 73.66 74.93 0)
 			(effects
@@
 			(project ""
 				(path "/e63e39d7-6ac0-4ffd-8aa3-1841a4541b55/90e1f016-3c60-4383-aa8d-def9977ac47b/78a99c0a-f468-453e-aea1-d254ed568110"
-					(reference "#PWR069")
-					(unit 1)
-				)
-				(path "/e63e39d7-6ac0-4ffd-8aa3-1841a4541b55/90e1f016-3c60-4383-aa8d-def9977ac47b/d909784a-ae31-4c8f-b386-03ea0f044fee"
-					(reference "#PWR078")
+					(reference "#PWR084")
+					(unit 1)
+				)
+				(path "/e63e39d7-6ac0-4ffd-8aa3-1841a4541b55/90e1f016-3c60-4383-aa8d-def9977ac47b/d909784a-ae31-4c8f-b386-03ea0f044fee"
+					(reference "#PWR093")
 					(unit 1)
 				)
@@
 		(on_board yes)
 		(dnp no)
-		(property "Reference" "#PWR074"
+		(property "Reference" "#PWR089"
 			(at 152.4 43.18 0)
 			(effects
@@
 			(project ""
 				(path "/e63e39d7-6ac0-4ffd-8aa3-1841a4541b55/90e1f016-3c60-4383-aa8d-def9977ac47b/78a99c0a-f468-453e-aea1-d254ed568110"
-					(reference "#PWR074")
-					(unit 1)
-				)
-				(path "/e63e39d7-6ac0-4ffd-8aa3-1841a4541b55/90e1f016-3c60-4383-aa8d-def9977ac47b/d909784a-ae31-4c8f-b386-03ea0f044fee"
-					(reference "#PWR083")
+					(reference "#PWR089")
+					(unit 1)
+				)
+				(path "/e63e39d7-6ac0-4ffd-8aa3-1841a4541b55/90e1f016-3c60-4383-aa8d-def9977ac47b/d909784a-ae31-4c8f-b386-03ea0f044fee"
+					(reference "#PWR098")
 					(unit 1)
 				)
@@
 		(dnp no)
 		(fields_autoplaced yes)
-		(property "Reference" "#PWR067"
+		(property "Reference" "#PWR082"
 			(at 33.02 77.47 0)
 			(effects
@@
 			(project ""
 				(path "/e63e39d7-6ac0-4ffd-8aa3-1841a4541b55/90e1f016-3c60-4383-aa8d-def9977ac47b/78a99c0a-f468-453e-aea1-d254ed568110"
-					(reference "#PWR067")
-					(unit 1)
-				)
-				(path "/e63e39d7-6ac0-4ffd-8aa3-1841a4541b55/90e1f016-3c60-4383-aa8d-def9977ac47b/d909784a-ae31-4c8f-b386-03ea0f044fee"
-					(reference "#PWR076")
+					(reference "#PWR082")
+					(unit 1)
+				)
+				(path "/e63e39d7-6ac0-4ffd-8aa3-1841a4541b55/90e1f016-3c60-4383-aa8d-def9977ac47b/d909784a-ae31-4c8f-b386-03ea0f044fee"
+					(reference "#PWR091")
 					(unit 1)
 				)
@@
 		(on_board yes)
 		(dnp no)
-		(property "Reference" "#PWR071"
+		(property "Reference" "#PWR086"
 			(at 99.06 43.18 0)
 			(effects
@@
 			(project ""
 				(path "/e63e39d7-6ac0-4ffd-8aa3-1841a4541b55/90e1f016-3c60-4383-aa8d-def9977ac47b/78a99c0a-f468-453e-aea1-d254ed568110"
-					(reference "#PWR071")
-					(unit 1)
-				)
-				(path "/e63e39d7-6ac0-4ffd-8aa3-1841a4541b55/90e1f016-3c60-4383-aa8d-def9977ac47b/d909784a-ae31-4c8f-b386-03ea0f044fee"
-					(reference "#PWR080")
+					(reference "#PWR086")
+					(unit 1)
+				)
+				(path "/e63e39d7-6ac0-4ffd-8aa3-1841a4541b55/90e1f016-3c60-4383-aa8d-def9977ac47b/d909784a-ae31-4c8f-b386-03ea0f044fee"
+					(reference "#PWR095")
 					(unit 1)
 				)
@@
 		(on_board yes)
 		(dnp no)
-		(property "Reference" "U15"
+		(property "Reference" "U16"
 			(at 41.148 76.708 90)
 			(effects
@@
 			(project "fnx51"
 				(path "/e63e39d7-6ac0-4ffd-8aa3-1841a4541b55/90e1f016-3c60-4383-aa8d-def9977ac47b/78a99c0a-f468-453e-aea1-d254ed568110"
-					(reference "U15")
-					(unit 1)
-				)
-				(path "/e63e39d7-6ac0-4ffd-8aa3-1841a4541b55/90e1f016-3c60-4383-aa8d-def9977ac47b/d909784a-ae31-4c8f-b386-03ea0f044fee"
-					(reference "U18")
+					(reference "U16")
+					(unit 1)
+				)
+				(path "/e63e39d7-6ac0-4ffd-8aa3-1841a4541b55/90e1f016-3c60-4383-aa8d-def9977ac47b/d909784a-ae31-4c8f-b386-03ea0f044fee"
+					(reference "U19")
 					(unit 1)
 				)
@@
 		(on_board yes)
 		(dnp no)
-		(property "Reference" "U16"
+		(property "Reference" "U17"
 			(at 91.948 76.708 90)
 			(effects
@@
 			(project "fnx51"
 				(path "/e63e39d7-6ac0-4ffd-8aa3-1841a4541b55/90e1f016-3c60-4383-aa8d-def9977ac47b/78a99c0a-f468-453e-aea1-d254ed568110"
-					(reference "U16")
-					(unit 1)
-				)
-				(path "/e63e39d7-6ac0-4ffd-8aa3-1841a4541b55/90e1f016-3c60-4383-aa8d-def9977ac47b/d909784a-ae31-4c8f-b386-03ea0f044fee"
-					(reference "U19")
+					(reference "U17")
+					(unit 1)
+				)
+				(path "/e63e39d7-6ac0-4ffd-8aa3-1841a4541b55/90e1f016-3c60-4383-aa8d-def9977ac47b/d909784a-ae31-4c8f-b386-03ea0f044fee"
+					(reference "U20")
 					(unit 1)
 				)
@@
 		(on_board yes)
 		(dnp no)
-		(property "Reference" "#PWR075"
+		(property "Reference" "#PWR090"
 			(at 175.26 74.93 0)
 			(effects
@@
 			(project ""
 				(path "/e63e39d7-6ac0-4ffd-8aa3-1841a4541b55/90e1f016-3c60-4383-aa8d-def9977ac47b/78a99c0a-f468-453e-aea1-d254ed568110"
-					(reference "#PWR075")
-					(unit 1)
-				)
-				(path "/e63e39d7-6ac0-4ffd-8aa3-1841a4541b55/90e1f016-3c60-4383-aa8d-def9977ac47b/d909784a-ae31-4c8f-b386-03ea0f044fee"
-					(reference "#PWR084")
+					(reference "#PWR090")
+					(unit 1)
+				)
+				(path "/e63e39d7-6ac0-4ffd-8aa3-1841a4541b55/90e1f016-3c60-4383-aa8d-def9977ac47b/d909784a-ae31-4c8f-b386-03ea0f044fee"
+					(reference "#PWR099")
 					(unit 1)
 				)
@@
 		(on_board yes)
 		(dnp no)
-		(property "Reference" "#PWR072"
+		(property "Reference" "#PWR087"
 			(at 124.46 74.93 0)
 			(effects
@@
 			(project ""
 				(path "/e63e39d7-6ac0-4ffd-8aa3-1841a4541b55/90e1f016-3c60-4383-aa8d-def9977ac47b/78a99c0a-f468-453e-aea1-d254ed568110"
-					(reference "#PWR072")
-					(unit 1)
-				)
-				(path "/e63e39d7-6ac0-4ffd-8aa3-1841a4541b55/90e1f016-3c60-4383-aa8d-def9977ac47b/d909784a-ae31-4c8f-b386-03ea0f044fee"
-					(reference "#PWR081")
-					(unit 1)
-				)
+					(reference "#PWR087")
+					(unit 1)
+				)
+				(path "/e63e39d7-6ac0-4ffd-8aa3-1841a4541b55/90e1f016-3c60-4383-aa8d-def9977ac47b/d909784a-ae31-4c8f-b386-03ea0f044fee"
+					(reference "#PWR096")
+					(unit 1)
+				)

Commit message: WIP schematic
Parts:
- renumbered U16 to U17, U17 to U18, U18 to U19
Changed lines of the file:
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@@
 		(dnp no)
 		(fields_autoplaced yes)
-		(property "Reference" "#PWR085"
+		(property "Reference" "#PWR0100"
 			(at 83.82 77.47 0)
 			(effects
@@
 			(project ""
 				(path "/e63e39d7-6ac0-4ffd-8aa3-1841a4541b55/90e1f016-3c60-4383-aa8d-def9977ac47b/78a99c0a-f468-453e-aea1-d254ed568110"
-					(reference "#PWR085")
-					(unit 1)
-				)
-				(path "/e63e39d7-6ac0-4ffd-8aa3-1841a4541b55/90e1f016-3c60-4383-aa8d-def9977ac47b/d909784a-ae31-4c8f-b386-03ea0f044fee"
-					(reference "#PWR094")
+					(reference "#PWR0100")
+					(unit 1)
+				)
+				(path "/e63e39d7-6ac0-4ffd-8aa3-1841a4541b55/90e1f016-3c60-4383-aa8d-def9977ac47b/d909784a-ae31-4c8f-b386-03ea0f044fee"
+					(reference "#PWR0109")
 					(unit 1)
 				)
@@
 		(on_board yes)
 		(dnp no)
-		(property "Reference" "#PWR083"
+		(property "Reference" "#PWR098"
 			(at 58.42 43.18 0)
 			(effects
@@
 			(project ""
 				(path "/e63e39d7-6ac0-4ffd-8aa3-1841a4541b55/90e1f016-3c60-4383-aa8d-def9977ac47b/78a99c0a-f468-453e-aea1-d254ed568110"
-					(reference "#PWR083")
-					(unit 1)
-				)
-				(path "/e63e39d7-6ac0-4ffd-8aa3-1841a4541b55/90e1f016-3c60-4383-aa8d-def9977ac47b/d909784a-ae31-4c8f-b386-03ea0f044fee"
-					(reference "#PWR092")
+					(reference "#PWR098")
+					(unit 1)
+				)
+				(path "/e63e39d7-6ac0-4ffd-8aa3-1841a4541b55/90e1f016-3c60-4383-aa8d-def9977ac47b/d909784a-ae31-4c8f-b386-03ea0f044fee"
+					(reference "#PWR0107")
 					(unit 1)
 				)
@@
 		(on_board yes)
 		(dnp no)
-		(property "Reference" "U18"
+		(property "Reference" "U19"
 			(at 142.748 76.708 90)
 			(effects
@@
 			(project ""
 				(path "/e63e39d7-6ac0-4ffd-8aa3-1841a4541b55/90e1f016-3c60-4383-aa8d-def9977ac47b/78a99c0a-f468-453e-aea1-d254ed568110"
-					(reference "U18")
-					(unit 1)
-				)
-				(path "/e63e39d7-6ac0-4ffd-8aa3-1841a4541b55/90e1f016-3c60-4383-aa8d-def9977ac47b/d909784a-ae31-4c8f-b386-03ea0f044fee"
-					(reference "U21")
+					(reference "U19")
+					(unit 1)
+				)
+				(path "/e63e39d7-6ac0-4ffd-8aa3-1841a4541b55/90e1f016-3c60-4383-aa8d-def9977ac47b/d909784a-ae31-4c8f-b386-03ea0f044fee"
+					(reference "U22")
 					(unit 1)
 				)
@@
 		(dnp no)
 		(fields_autoplaced yes)
-		(property "Reference" "#PWR088"
+		(property "Reference" "#PWR0103"
 			(at 134.62 77.47 0)
 			(effects
@@
 			(project ""
 				(path "/e63e39d7-6ac0-4ffd-8aa3-1841a4541b55/90e1f016-3c60-4383-aa8d-def9977ac47b/78a99c0a-f468-453e-aea1-d254ed568110"
-					(reference "#PWR088")
-					(unit 1)
-				)
-				(path "/e63e39d7-6ac0-4ffd-8aa3-1841a4541b55/90e1f016-3c60-4383-aa8d-def9977ac47b/d909784a-ae31-4c8f-b386-03ea0f044fee"
-					(reference "#PWR097")
+					(reference "#PWR0103")
+					(unit 1)
+				)
+				(path "/e63e39d7-6ac0-4ffd-8aa3-1841a4541b55/90e1f016-3c60-4383-aa8d-def9977ac47b/d909784a-ae31-4c8f-b386-03ea0f044fee"
+					(reference "#PWR0112")
 					(unit 1)
 				)
@@
 		(on_board yes)
 		(dnp no)
-		(property "Reference" "#PWR084"
+		(property "Reference" "#PWR099"
 			(at 73.66 74.93 0)
 			(effects
@@
 			(project ""
 				(path "/e63e39d7-6ac0-4ffd-8aa3-1841a4541b55/90e1f016-3c60-4383-aa8d-def9977ac47b/78a99c0a-f468-453e-aea1-d254ed568110"
-					(reference "#PWR084")
-					(unit 1)
-				)
-				(path "/e63e39d7-6ac0-4ffd-8aa3-1841a4541b55/90e1f016-3c60-4383-aa8d-def9977ac47b/d909784a-ae31-4c8f-b386-03ea0f044fee"
-					(reference "#PWR093")
+					(reference "#PWR099")
+					(unit 1)
+				)
+				(path "/e63e39d7-6ac0-4ffd-8aa3-1841a4541b55/90e1f016-3c60-4383-aa8d-def9977ac47b/d909784a-ae31-4c8f-b386-03ea0f044fee"
+					(reference "#PWR0108")
 					(unit 1)
 				)
@@
 		(on_board yes)
 		(dnp no)
-		(property "Reference" "#PWR089"
+		(property "Reference" "#PWR0104"
 			(at 152.4 43.18 0)
 			(effects
@@
 			(project ""
 				(path "/e63e39d7-6ac0-4ffd-8aa3-1841a4541b55/90e1f016-3c60-4383-aa8d-def9977ac47b/78a99c0a-f468-453e-aea1-d254ed568110"
-					(reference "#PWR089")
-					(unit 1)
-				)
-				(path "/e63e39d7-6ac0-4ffd-8aa3-1841a4541b55/90e1f016-3c60-4383-aa8d-def9977ac47b/d909784a-ae31-4c8f-b386-03ea0f044fee"
-					(reference "#PWR098")
+					(reference "#PWR0104")
+					(unit 1)
+				)
+				(path "/e63e39d7-6ac0-4ffd-8aa3-1841a4541b55/90e1f016-3c60-4383-aa8d-def9977ac47b/d909784a-ae31-4c8f-b386-03ea0f044fee"
+					(reference "#PWR0113")
 					(unit 1)
 				)
@@
 		(dnp no)
 		(fields_autoplaced yes)
-		(property "Reference" "#PWR082"
+		(property "Reference" "#PWR097"
 			(at 33.02 77.47 0)
 			(effects
@@
 			(project ""
 				(path "/e63e39d7-6ac0-4ffd-8aa3-1841a4541b55/90e1f016-3c60-4383-aa8d-def9977ac47b/78a99c0a-f468-453e-aea1-d254ed568110"
-					(reference "#PWR082")
-					(unit 1)
-				)
-				(path "/e63e39d7-6ac0-4ffd-8aa3-1841a4541b55/90e1f016-3c60-4383-aa8d-def9977ac47b/d909784a-ae31-4c8f-b386-03ea0f044fee"
-					(reference "#PWR091")
+					(reference "#PWR097")
+					(unit 1)
+				)
+				(path "/e63e39d7-6ac0-4ffd-8aa3-1841a4541b55/90e1f016-3c60-4383-aa8d-def9977ac47b/d909784a-ae31-4c8f-b386-03ea0f044fee"
+					(reference "#PWR0106")
 					(unit 1)
 				)
@@
 		(on_board yes)
 		(dnp no)
-		(property "Reference" "#PWR086"
+		(property "Reference" "#PWR0101"
 			(at 99.06 43.18 0)
 			(effects
@@
 			(project ""
 				(path "/e63e39d7-6ac0-4ffd-8aa3-1841a4541b55/90e1f016-3c60-4383-aa8d-def9977ac47b/78a99c0a-f468-453e-aea1-d254ed568110"
-					(reference "#PWR086")
-					(unit 1)
-				)
-				(path "/e63e39d7-6ac0-4ffd-8aa3-1841a4541b55/90e1f016-3c60-4383-aa8d-def9977ac47b/d909784a-ae31-4c8f-b386-03ea0f044fee"
-					(reference "#PWR095")
+					(reference "#PWR0101")
+					(unit 1)
+				)
+				(path "/e63e39d7-6ac0-4ffd-8aa3-1841a4541b55/90e1f016-3c60-4383-aa8d-def9977ac47b/d909784a-ae31-4c8f-b386-03ea0f044fee"
+					(reference "#PWR0110")
 					(unit 1)
 				)
@@
 		(on_board yes)
 		(dnp no)
-		(property "Reference" "U16"
+		(property "Reference" "U17"
 			(at 41.148 76.708 90)
 			(effects
@@
 			(project "fnx51"
 				(path "/e63e39d7-6ac0-4ffd-8aa3-1841a4541b55/90e1f016-3c60-4383-aa8d-def9977ac47b/78a99c0a-f468-453e-aea1-d254ed568110"
-					(reference "U16")
-					(unit 1)
-				)
-				(path "/e63e39d7-6ac0-4ffd-8aa3-1841a4541b55/90e1f016-3c60-4383-aa8d-def9977ac47b/d909784a-ae31-4c8f-b386-03ea0f044fee"
-					(reference "U19")
+					(reference "U17")
+					(unit 1)
+				)
+				(path "/e63e39d7-6ac0-4ffd-8aa3-1841a4541b55/90e1f016-3c60-4383-aa8d-def9977ac47b/d909784a-ae31-4c8f-b386-03ea0f044fee"
+					(reference "U20")
 					(unit 1)
 				)
@@
 		(on_board yes)
 		(dnp no)
-		(property "Reference" "U17"
+		(property "Reference" "U18"
 			(at 91.948 76.708 90)
 			(effects
@@
 			(project "fnx51"
 				(path "/e63e39d7-6ac0-4ffd-8aa3-1841a4541b55/90e1f016-3c60-4383-aa8d-def9977ac47b/78a99c0a-f468-453e-aea1-d254ed568110"
-					(reference "U17")
-					(unit 1)
-				)
-				(path "/e63e39d7-6ac0-4ffd-8aa3-1841a4541b55/90e1f016-3c60-4383-aa8d-def9977ac47b/d909784a-ae31-4c8f-b386-03ea0f044fee"
-					(reference "U20")
+					(reference "U18")
+					(unit 1)
+				)
+				(path "/e63e39d7-6ac0-4ffd-8aa3-1841a4541b55/90e1f016-3c60-4383-aa8d-def9977ac47b/d909784a-ae31-4c8f-b386-03ea0f044fee"
+					(reference "U21")
 					(unit 1)
 				)
@@
 		(on_board yes)
 		(dnp no)
-		(property "Reference" "#PWR090"
+		(property "Reference" "#PWR0105"
 			(at 175.26 74.93 0)
 			(effects
@@
 			(project ""
 				(path "/e63e39d7-6ac0-4ffd-8aa3-1841a4541b55/90e1f016-3c60-4383-aa8d-def9977ac47b/78a99c0a-f468-453e-aea1-d254ed568110"
-					(reference "#PWR090")
-					(unit 1)
-				)
-				(path "/e63e39d7-6ac0-4ffd-8aa3-1841a4541b55/90e1f016-3c60-4383-aa8d-def9977ac47b/d909784a-ae31-4c8f-b386-03ea0f044fee"
-					(reference "#PWR099")
+					(reference "#PWR0105")
+					(unit 1)
+				)
+				(path "/e63e39d7-6ac0-4ffd-8aa3-1841a4541b55/90e1f016-3c60-4383-aa8d-def9977ac47b/d909784a-ae31-4c8f-b386-03ea0f044fee"
+					(reference "#PWR0114")
 					(unit 1)
 				)
@@
 		(on_board yes)
 		(dnp no)
-		(property "Reference" "#PWR087"
+		(property "Reference" "#PWR0102"
 			(at 124.46 74.93 0)
 			(effects
@@
 			(project ""
 				(path "/e63e39d7-6ac0-4ffd-8aa3-1841a4541b55/90e1f016-3c60-4383-aa8d-def9977ac47b/78a99c0a-f468-453e-aea1-d254ed568110"
-					(reference "#PWR087")
-					(unit 1)
-				)
-				(path "/e63e39d7-6ac0-4ffd-8aa3-1841a4541b55/90e1f016-3c60-4383-aa8d-def9977ac47b/d909784a-ae31-4c8f-b386-03ea0f044fee"
-					(reference "#PWR096")
-					(unit 1)
-				)
+					(reference "#PWR0102")
+					(unit 1)
+				)
+				(path "/e63e39d7-6ac0-4ffd-8aa3-1841a4541b55/90e1f016-3c60-4383-aa8d-def9977ac47b/d909784a-ae31-4c8f-b386-03ea0f044fee"
+					(reference "#PWR0111")
+					(unit 1)
+				)

Commit message: WIP PCB (add bypass caps, minor fixes)
Parts:
- added C24, C25, C26: 100nF, symbol Device:C_Small
- renumbered U17 to U19, U18 to U20, U19 to U21
Connections:
- net +5V: now also C24.2, C25.2, C26.2
- net GND: now also C24.1, C25.1, C26.1
Other:
- moved on the sheet: U19, U20, U21
