File: pcb/comp_ff.kicad_sch (KiCad schematic)
At the start: 4 parts

Commit message: WIP schematic
Parts:
- gave numbers to parts that had none: 4
Connections:
- net VCC renamed +5V
Changed lines of the file:
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@@
 		(dnp no)
 		(fields_autoplaced yes)
-		(property "Reference" "U?"
+		(property "Reference" "U20"
 			(at 108.8741 91.44 0)
 			(effects
@@
 			(project ""
 				(path "/e63e39d7-6ac0-4ffd-8aa3-1841a4541b55/90e1f016-3c60-4383-aa8d-def9977ac47b/080e9e7b-a3e6-4d7b-a91a-d4d1bce9fcbf"
-					(reference "U?")
+					(reference "U20")
 					(unit 1)
 				)
 				(path "/e63e39d7-6ac0-4ffd-8aa3-1841a4541b55/90e1f016-3c60-4383-aa8d-def9977ac47b/0e21d398-15c6-48fd-a9a5-1cc9fd257aa3"
-					(reference "U?")
+					(reference "U27")
 					(unit 1)
 				)
 				(path "/e63e39d7-6ac0-4ffd-8aa3-1841a4541b55/90e1f016-3c60-4383-aa8d-def9977ac47b/763856e2-a839-4490-96d3-1a5f6bf03d10"
-					(reference "U?")
+					(reference "U23")
 					(unit 1)
 				)
 				(path "/e63e39d7-6ac0-4ffd-8aa3-1841a4541b55/90e1f016-3c60-4383-aa8d-def9977ac47b/be7e522f-a717-4004-b2b4-d0582d753e6f"
-					(reference "U?")
+					(reference "U30")
 					(unit 1)
 				)
@@
 		(on_board yes)
 		(dnp no)
-		(property "Reference" "#PWR?"
+		(property "Reference" "#PWR075"
 			(at 71.12 163.83 0)
 			(effects
@@
 			(project "fnx51"
 				(path "/e63e39d7-6ac0-4ffd-8aa3-1841a4541b55/90e1f016-3c60-4383-aa8d-def9977ac47b/080e9e7b-a3e6-4d7b-a91a-d4d1bce9fcbf"
-					(reference "#PWR?")
+					(reference "#PWR075")
 					(unit 1)
 				)
 				(path "/e63e39d7-6ac0-4ffd-8aa3-1841a4541b55/90e1f016-3c60-4383-aa8d-def9977ac47b/0e21d398-15c6-48fd-a9a5-1cc9fd257aa3"
-					(reference "#PWR?")
+					(reference "#PWR085")
 					(unit 1)
 				)
 				(path "/e63e39d7-6ac0-4ffd-8aa3-1841a4541b55/90e1f016-3c60-4383-aa8d-def9977ac47b/763856e2-a839-4490-96d3-1a5f6bf03d10"
-					(reference "#PWR?")
+					(reference "#PWR080")
 					(unit 1)
 				)
 				(path "/e63e39d7-6ac0-4ffd-8aa3-1841a4541b55/90e1f016-3c60-4383-aa8d-def9977ac47b/be7e522f-a717-4004-b2b4-d0582d753e6f"
-					(reference "#PWR?")
+					(reference "#PWR090")
 					(unit 1)
 				)
@@
 		(on_board yes)
 		(dnp no)
-		(property "Reference" "U?"
+		(property "Reference" "U18"
 			(at 64.77 24.13 0)
 			(effects
@@
 			(project ""
 				(path "/e63e39d7-6ac0-4ffd-8aa3-1841a4541b55/90e1f016-3c60-4383-aa8d-def9977ac47b/080e9e7b-a3e6-4d7b-a91a-d4d1bce9fcbf"
-					(reference "U?")
+					(reference "U18")
 					(unit 1)
 				)
 				(path "/e63e39d7-6ac0-4ffd-8aa3-1841a4541b55/90e1f016-3c60-4383-aa8d-def9977ac47b/0e21d398-15c6-48fd-a9a5-1cc9fd257aa3"
-					(reference "U?")
+					(reference "U24")
 					(unit 1)
 				)
 				(path "/e63e39d7-6ac0-4ffd-8aa3-1841a4541b55/90e1f016-3c60-4383-aa8d-def9977ac47b/763856e2-a839-4490-96d3-1a5f6bf03d10"
-					(reference "U?")
+					(reference "U21")
 					(unit 1)
 				)
 				(path "/e63e39d7-6ac0-4ffd-8aa3-1841a4541b55/90e1f016-3c60-4383-aa8d-def9977ac47b/be7e522f-a717-4004-b2b4-d0582d753e6f"
-					(reference "U?")
+					(reference "U28")
 					(unit 1)
 				)
@@
 		(on_board yes)
 		(dnp no)
-		(property "Reference" "#PWR?"
+		(property "Reference" "#PWR073"
 			(at 71.12 87.63 0)
 			(effects
@@
 			(project ""
 				(path "/e63e39d7-6ac0-4ffd-8aa3-1841a4541b55/90e1f016-3c60-4383-aa8d-def9977ac47b/080e9e7b-a3e6-4d7b-a91a-d4d1bce9fcbf"
-					(reference "#PWR?")
+					(reference "#PWR073")
 					(unit 1)
 				)
 				(path "/e63e39d7-6ac0-4ffd-8aa3-1841a4541b55/90e1f016-3c60-4383-aa8d-def9977ac47b/0e21d398-15c6-48fd-a9a5-1cc9fd257aa3"
-					(reference "#PWR?")
+					(reference "#PWR083")
 					(unit 1)
 				)
 				(path "/e63e39d7-6ac0-4ffd-8aa3-1841a4541b55/90e1f016-3c60-4383-aa8d-def9977ac47b/763856e2-a839-4490-96d3-1a5f6bf03d10"
-					(reference "#PWR?")
+					(reference "#PWR078")
 					(unit 1)
 				)
 				(path "/e63e39d7-6ac0-4ffd-8aa3-1841a4541b55/90e1f016-3c60-4383-aa8d-def9977ac47b/be7e522f-a717-4004-b2b4-d0582d753e6f"
-					(reference "#PWR?")
+					(reference "#PWR088")
 					(unit 1)
 				)
@@
 		(on_board yes)
 		(dnp no)
-		(property "Reference" "U?"
+		(property "Reference" "U19"
 			(at 64.77 100.33 0)
 			(effects
@@
 			(project "fnx51"
 				(path "/e63e39d7-6ac0-4ffd-8aa3-1841a4541b55/90e1f016-3c60-4383-aa8d-def9977ac47b/080e9e7b-a3e6-4d7b-a91a-d4d1bce9fcbf"
-					(reference "U?")
+					(reference "U19")
 					(unit 1)
 				)
 				(path "/e63e39d7-6ac0-4ffd-8aa3-1841a4541b55/90e1f016-3c60-4383-aa8d-def9977ac47b/0e21d398-15c6-48fd-a9a5-1cc9fd257aa3"
-					(reference "U?")
+					(reference "U25")
 					(unit 1)
 				)
 				(path "/e63e39d7-6ac0-4ffd-8aa3-1841a4541b55/90e1f016-3c60-4383-aa8d-def9977ac47b/763856e2-a839-4490-96d3-1a5f6bf03d10"
-					(reference "U?")
+					(reference "U22")
 					(unit 1)
 				)
 				(path "/e63e39d7-6ac0-4ffd-8aa3-1841a4541b55/90e1f016-3c60-4383-aa8d-def9977ac47b/be7e522f-a717-4004-b2b4-d0582d753e6f"
-					(reference "U?")
+					(reference "U29")
 					(unit 1)
 				)
@@
 	)
 	(symbol
-		(lib_id "power:VCC")
+		(lib_id "power:+5V")
 		(at 106.68 93.98 0)
 		(unit 1)
@@
 		(dnp no)
 		(fields_autoplaced yes)
-		(property "Reference" "#PWR?"
+		(property "Reference" "#PWR076"
 			(at 106.68 97.79 0)
 			(effects
@@
 			)
 		)
-		(property "Value" "VCC"
-			(at 106.68 88.9 0)
-			(effects
-				(font
-					(size 1.27 1.27)
-				)
+		(property "Value" "+5V"
+			(at 109.22 92.7099 0)
+			(effects
+				(font
+					(size 1.27 1.27)
+				)
+				(justify left)
 			)
 		)
@@
 			)
 		)
-		(property "Description" "Power symbol creates a global label with name \"VCC\""
+		(property "Description" "Power symbol creates a global label with name \"+5V\""
 			(at 106.68 93.98 0)
 			(effects
@@
 			(project ""
 				(path "/e63e39d7-6ac0-4ffd-8aa3-1841a4541b55/90e1f016-3c60-4383-aa8d-def9977ac47b/080e9e7b-a3e6-4d7b-a91a-d4d1bce9fcbf"
-					(reference "#PWR?")
+					(reference "#PWR076")
 					(unit 1)
 				)
 				(path "/e63e39d7-6ac0-4ffd-8aa3-1841a4541b55/90e1f016-3c60-4383-aa8d-def9977ac47b/0e21d398-15c6-48fd-a9a5-1cc9fd257aa3"
-					(reference "#PWR?")
+					(reference "#PWR086")
 					(unit 1)
 				)
 				(path "/e63e39d7-6ac0-4ffd-8aa3-1841a4541b55/90e1f016-3c60-4383-aa8d-def9977ac47b/763856e2-a839-4490-96d3-1a5f6bf03d10"
-					(reference "#PWR?")
+					(reference "#PWR081")
 					(unit 1)
 				)
 				(path "/e63e39d7-6ac0-4ffd-8aa3-1841a4541b55/90e1f016-3c60-4383-aa8d-def9977ac47b/be7e522f-a717-4004-b2b4-d0582d753e6f"
-					(reference "#PWR?")
+					(reference "#PWR091")
 					(unit 1)
 				)
@@
 	)
 	(symbol
-		(lib_id "power:VCC")
+		(lib_id "power:+5V")
 		(at 71.12 20.32 0)
 		(unit 1)
@@
 		(on_board yes)
 		(dnp no)
-		(property "Reference" "#PWR?"
+		(property "Reference" "#PWR072"
 			(at 71.12 24.13 0)
 			(effects
@@
 			)
 		)
-		(property "Value" "VCC"
+		(property "Value" "+5V"
 			(at 71.12 16.51 0)
 			(effects
@@
 			)
 		)
-		(property "Description" "Power symbol creates a global label with name \"VCC\""
+		(property "Description" "Power symbol creates a global label with name \"+5V\""
 			(at 71.12 20.32 0)
 			(effects
@@
 			(project ""
 				(path "/e63e39d7-6ac0-4ffd-8aa3-1841a4541b55/90e1f016-3c60-4383-aa8d-def9977ac47b/080e9e7b-a3e6-4d7b-a91a-d4d1bce9fcbf"
-					(reference "#PWR?")
+					(reference "#PWR072")
 					(unit 1)
 				)
 				(path "/e63e39d7-6ac0-4ffd-8aa3-1841a4541b55/90e1f016-3c60-4383-aa8d-def9977ac47b/0e21d398-15c6-48fd-a9a5-1cc9fd257aa3"
-					(reference "#PWR?")
+					(reference "#PWR082")
 					(unit 1)
 				)
 				(path "/e63e39d7-6ac0-4ffd-8aa3-1841a4541b55/90e1f016-3c60-4383-aa8d-def9977ac47b/763856e2-a839-4490-96d3-1a5f6bf03d10"
-					(reference "#PWR?")
+					(reference "#PWR077")
 					(unit 1)
 				)
 				(path "/e63e39d7-6ac0-4ffd-8aa3-1841a4541b55/90e1f016-3c60-4383-aa8d-def9977ac47b/be7e522f-a717-4004-b2b4-d0582d753e6f"
-					(reference "#PWR?")
+					(reference "#PWR087")
 					(unit 1)
 				)
@@
 	)
 	(symbol
-		(lib_id "power:VCC")
+		(lib_id "power:+5V")
 		(at 71.12 96.52 0)
 		(unit 1)
@@
 		(on_board yes)
 		(dnp no)
-		(property "Reference" "#PWR?"
+		(property "Reference" "#PWR074"
 			(at 71.12 100.33 0)
 			(effects
@@
 			)
 		)
-		(property "Value" "VCC"
+		(property "Value" "+5V"
 			(at 71.12 92.71 0)
 			(effects
@@
 			)
 		)
-		(property "Description" "Power symbol creates a global label with name \"VCC\""
+		(property "Description" "Power symbol creates a global label with name \"+5V\""
 			(at 71.12 96.52 0)
 			(effects
@@
 			(project "fnx51"
 				(path "/e63e39d7-6ac0-4ffd-8aa3-1841a4541b55/90e1f016-3c60-4383-aa8d-def9977ac47b/080e9e7b-a3e6-4d7b-a91a-d4d1bce9fcbf"
-					(reference "#PWR?")
+					(reference "#PWR074")
 					(unit 1)
 				)
 				(path "/e63e39d7-6ac0-4ffd-8aa3-1841a4541b55/90e1f016-3c60-4383-aa8d-def9977ac47b/0e21d398-15c6-48fd-a9a5-1cc9fd257aa3"
-					(reference "#PWR?")
+					(reference "#PWR084")
 					(unit 1)
 				)
 				(path "/e63e39d7-6ac0-4ffd-8aa3-1841a4541b55/90e1f016-3c60-4383-aa8d-def9977ac47b/763856e2-a839-4490-96d3-1a5f6bf03d10"
-					(reference "#PWR?")
+					(reference "#PWR079")
 					(unit 1)
 				)
 				(path "/e63e39d7-6ac0-4ffd-8aa3-1841a4541b55/90e1f016-3c60-4383-aa8d-def9977ac47b/be7e522f-a717-4004-b2b4-d0582d753e6f"
-					(reference "#PWR?")
+					(reference "#PWR089")
 					(unit 1)
 				)
@@
 		(dnp no)
 		(fields_autoplaced yes)
-		(property "Reference" "U?"
+		(property "Reference" "U9"
 			(at 93.98 55.8799 90)
 			(effects
@@
 			(project ""
 				(path "/e63e39d7-6ac0-4ffd-8aa3-1841a4541b55/90e1f016-3c60-4383-aa8d-def9977ac47b/080e9e7b-a3e6-4d7b-a91a-d4d1bce9fcbf"
-					(reference "U?")
+					(reference "U9")
 					(unit 5)
 				)
 				(path "/e63e39d7-6ac0-4ffd-8aa3-1841a4541b55/90e1f016-3c60-4383-aa8d-def9977ac47b/0e21d398-15c6-48fd-a9a5-1cc9fd257aa3"
-					(reference "U?")
+					(reference "U26")
 					(unit 5)
 				)
 				(path "/e63e39d7-6ac0-4ffd-8aa3-1841a4541b55/90e1f016-3c60-4383-aa8d-def9977ac47b/763856e2-a839-4490-96d3-1a5f6bf03d10"
-					(reference "U?")
+					(reference "U9")
 					(unit 4)
 				)
 				(path "/e63e39d7-6ac0-4ffd-8aa3-1841a4541b55/90e1f016-3c60-4383-aa8d-def9977ac47b/be7e522f-a717-4004-b2b4-d0582d753e6f"
-					(reference "U?")
+					(reference "U9")
 					(unit 6)
 				)

Commit message: WIP PCB
Parts:
- renumbered U20 to U?, U18 to U?, U19 to U?, U9 to U?

Commit message: wip schematic
Parts:
- U?: value 74LS109 -> 74HC109
Connections:
- net at U?.2 (J): now also U?.2; no longer U?.10
- net at U?.19 (P=R): now also U?.1; no longer U?.11
Changed lines of the file:
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@@
 			)
 		)
-		(property "Value" "74LS109"
+		(property "Value" "74HC109"
 			(at 108.8741 93.98 0)
 			(effects
@@
 				(path "/e63e39d7-6ac0-4ffd-8aa3-1841a4541b55/90e1f016-3c60-4383-aa8d-def9977ac47b/763856e2-a839-4490-96d3-1a5f6bf03d10"
 					(reference "U?")
-					(unit 1)
-				)
-				(path "/e63e39d7-6ac0-4ffd-8aa3-1841a4541b55/90e1f016-3c60-4383-aa8d-def9977ac47b/be7e522f-a717-4004-b2b4-d0582d753e6f"
-					(reference "U?")
-					(unit 1)
+					(unit 2)
+				)
+				(path "/e63e39d7-6ac0-4ffd-8aa3-1841a4541b55/90e1f016-3c60-4383-aa8d-def9977ac47b/be7e522f-a717-4004-b2b4-d0582d753e6f"
+					(reference "U?")
+					(unit 2)
 				)
 			)
@@
 		(on_board yes)
 		(dnp no)
-		(fields_autoplaced yes)
 		(property "Reference" "#PWR?"
 			(at 106.68 97.79 0)
@@
 		)
 		(property "Value" "+5V"
-			(at 109.22 92.7099 0)
+			(at 104.14 88.9 0)
 			(effects
 				(font
@@
 		(lib_id "74xx:74HC04")
 		(at 88.9 57.15 270)
-		(unit 5)
+		(unit 1)
 		(exclude_from_sim no)
 		(in_bom yes)
@@
 				(path "/e63e39d7-6ac0-4ffd-8aa3-1841a4541b55/90e1f016-3c60-4383-aa8d-def9977ac47b/080e9e7b-a3e6-4d7b-a91a-d4d1bce9fcbf"
 					(reference "U?")
-					(unit 5)
-				)
-				(path "/e63e39d7-6ac0-4ffd-8aa3-1841a4541b55/90e1f016-3c60-4383-aa8d-def9977ac47b/0e21d398-15c6-48fd-a9a5-1cc9fd257aa3"
-					(reference "U?")
-					(unit 5)
-				)
-				(path "/e63e39d7-6ac0-4ffd-8aa3-1841a4541b55/90e1f016-3c60-4383-aa8d-def9977ac47b/763856e2-a839-4490-96d3-1a5f6bf03d10"
+					(unit 1)
+				)
+				(path "/e63e39d7-6ac0-4ffd-8aa3-1841a4541b55/90e1f016-3c60-4383-aa8d-def9977ac47b/0e21d398-15c6-48fd-a9a5-1cc9fd257aa3"
+					(reference "U?")
+					(unit 3)
+				)
+				(path "/e63e39d7-6ac0-4ffd-8aa3-1841a4541b55/90e1f016-3c60-4383-aa8d-def9977ac47b/763856e2-a839-4490-96d3-1a5f6bf03d10"
+					(reference "U?")
+					(unit 2)
+				)
+				(path "/e63e39d7-6ac0-4ffd-8aa3-1841a4541b55/90e1f016-3c60-4383-aa8d-def9977ac47b/be7e522f-a717-4004-b2b4-d0582d753e6f"
 					(reference "U?")
 					(unit 4)
 				)
-				(path "/e63e39d7-6ac0-4ffd-8aa3-1841a4541b55/90e1f016-3c60-4383-aa8d-def9977ac47b/be7e522f-a717-4004-b2b4-d0582d753e6f"
-					(reference "U?")
-					(unit 6)
-				)
-			)
+			)
