File: pcb/comp_ff.kicad_sch (KiCad schematic)
At the start: 4 parts, among them U22 74HC688, U23 74HC688, U24 74HC04, U25 74HC109

Commit message: WIP schematic
Parts:
- renumbered U24 to U15, U22 to U23, U23 to U24
Changed lines of the file:
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@@
 		(on_board yes)
 		(dnp no)
-		(property "Reference" "#PWR0103"
+		(property "Reference" "#PWR0118"
 			(at 71.12 163.83 0)
 			(effects
@@
 			(project "fnx51"
 				(path "/e63e39d7-6ac0-4ffd-8aa3-1841a4541b55/90e1f016-3c60-4383-aa8d-def9977ac47b/080e9e7b-a3e6-4d7b-a91a-d4d1bce9fcbf"
-					(reference "#PWR0103")
-					(unit 1)
-				)
-				(path "/e63e39d7-6ac0-4ffd-8aa3-1841a4541b55/90e1f016-3c60-4383-aa8d-def9977ac47b/0e21d398-15c6-48fd-a9a5-1cc9fd257aa3"
-					(reference "#PWR0113")
-					(unit 1)
-				)
-				(path "/e63e39d7-6ac0-4ffd-8aa3-1841a4541b55/90e1f016-3c60-4383-aa8d-def9977ac47b/763856e2-a839-4490-96d3-1a5f6bf03d10"
-					(reference "#PWR0108")
-					(unit 1)
-				)
-				(path "/e63e39d7-6ac0-4ffd-8aa3-1841a4541b55/90e1f016-3c60-4383-aa8d-def9977ac47b/be7e522f-a717-4004-b2b4-d0582d753e6f"
 					(reference "#PWR0118")
+					(unit 1)
+				)
+				(path "/e63e39d7-6ac0-4ffd-8aa3-1841a4541b55/90e1f016-3c60-4383-aa8d-def9977ac47b/0e21d398-15c6-48fd-a9a5-1cc9fd257aa3"
+					(reference "#PWR0128")
+					(unit 1)
+				)
+				(path "/e63e39d7-6ac0-4ffd-8aa3-1841a4541b55/90e1f016-3c60-4383-aa8d-def9977ac47b/763856e2-a839-4490-96d3-1a5f6bf03d10"
+					(reference "#PWR0123")
+					(unit 1)
+				)
+				(path "/e63e39d7-6ac0-4ffd-8aa3-1841a4541b55/90e1f016-3c60-4383-aa8d-def9977ac47b/be7e522f-a717-4004-b2b4-d0582d753e6f"
+					(reference "#PWR0133")
 					(unit 1)
 				)
@@
 		(on_board yes)
 		(dnp no)
-		(property "Reference" "U22"
+		(property "Reference" "U23"
 			(at 64.77 24.13 0)
 			(effects
@@
 			(project ""
 				(path "/e63e39d7-6ac0-4ffd-8aa3-1841a4541b55/90e1f016-3c60-4383-aa8d-def9977ac47b/080e9e7b-a3e6-4d7b-a91a-d4d1bce9fcbf"
-					(reference "U22")
+					(reference "U23")
 					(unit 1)
 				)
@@
 		(on_board yes)
 		(dnp no)
-		(property "Reference" "#PWR0101"
+		(property "Reference" "#PWR0116"
 			(at 71.12 87.63 0)
 			(effects
@@
 			(project ""
 				(path "/e63e39d7-6ac0-4ffd-8aa3-1841a4541b55/90e1f016-3c60-4383-aa8d-def9977ac47b/080e9e7b-a3e6-4d7b-a91a-d4d1bce9fcbf"
-					(reference "#PWR0101")
-					(unit 1)
-				)
-				(path "/e63e39d7-6ac0-4ffd-8aa3-1841a4541b55/90e1f016-3c60-4383-aa8d-def9977ac47b/0e21d398-15c6-48fd-a9a5-1cc9fd257aa3"
-					(reference "#PWR0111")
-					(unit 1)
-				)
-				(path "/e63e39d7-6ac0-4ffd-8aa3-1841a4541b55/90e1f016-3c60-4383-aa8d-def9977ac47b/763856e2-a839-4490-96d3-1a5f6bf03d10"
-					(reference "#PWR0106")
-					(unit 1)
-				)
-				(path "/e63e39d7-6ac0-4ffd-8aa3-1841a4541b55/90e1f016-3c60-4383-aa8d-def9977ac47b/be7e522f-a717-4004-b2b4-d0582d753e6f"
 					(reference "#PWR0116")
+					(unit 1)
+				)
+				(path "/e63e39d7-6ac0-4ffd-8aa3-1841a4541b55/90e1f016-3c60-4383-aa8d-def9977ac47b/0e21d398-15c6-48fd-a9a5-1cc9fd257aa3"
+					(reference "#PWR0126")
+					(unit 1)
+				)
+				(path "/e63e39d7-6ac0-4ffd-8aa3-1841a4541b55/90e1f016-3c60-4383-aa8d-def9977ac47b/763856e2-a839-4490-96d3-1a5f6bf03d10"
+					(reference "#PWR0121")
+					(unit 1)
+				)
+				(path "/e63e39d7-6ac0-4ffd-8aa3-1841a4541b55/90e1f016-3c60-4383-aa8d-def9977ac47b/be7e522f-a717-4004-b2b4-d0582d753e6f"
+					(reference "#PWR0131")
 					(unit 1)
 				)
@@
 		(on_board yes)
 		(dnp no)
-		(property "Reference" "U23"
+		(property "Reference" "U24"
 			(at 64.77 100.33 0)
 			(effects
@@
 			(project "fnx51"
 				(path "/e63e39d7-6ac0-4ffd-8aa3-1841a4541b55/90e1f016-3c60-4383-aa8d-def9977ac47b/080e9e7b-a3e6-4d7b-a91a-d4d1bce9fcbf"
-					(reference "U23")
+					(reference "U24")
 					(unit 1)
 				)
@@
 		(on_board yes)
 		(dnp no)
-		(property "Reference" "#PWR0104"
+		(property "Reference" "#PWR0119"
 			(at 106.68 97.79 0)
 			(effects
@@
 			(project ""
 				(path "/e63e39d7-6ac0-4ffd-8aa3-1841a4541b55/90e1f016-3c60-4383-aa8d-def9977ac47b/080e9e7b-a3e6-4d7b-a91a-d4d1bce9fcbf"
-					(reference "#PWR0104")
-					(unit 1)
-				)
-				(path "/e63e39d7-6ac0-4ffd-8aa3-1841a4541b55/90e1f016-3c60-4383-aa8d-def9977ac47b/0e21d398-15c6-48fd-a9a5-1cc9fd257aa3"
-					(reference "#PWR0114")
-					(unit 1)
-				)
-				(path "/e63e39d7-6ac0-4ffd-8aa3-1841a4541b55/90e1f016-3c60-4383-aa8d-def9977ac47b/763856e2-a839-4490-96d3-1a5f6bf03d10"
-					(reference "#PWR0109")
-					(unit 1)
-				)
-				(path "/e63e39d7-6ac0-4ffd-8aa3-1841a4541b55/90e1f016-3c60-4383-aa8d-def9977ac47b/be7e522f-a717-4004-b2b4-d0582d753e6f"
 					(reference "#PWR0119")
+					(unit 1)
+				)
+				(path "/e63e39d7-6ac0-4ffd-8aa3-1841a4541b55/90e1f016-3c60-4383-aa8d-def9977ac47b/0e21d398-15c6-48fd-a9a5-1cc9fd257aa3"
+					(reference "#PWR0129")
+					(unit 1)
+				)
+				(path "/e63e39d7-6ac0-4ffd-8aa3-1841a4541b55/90e1f016-3c60-4383-aa8d-def9977ac47b/763856e2-a839-4490-96d3-1a5f6bf03d10"
+					(reference "#PWR0124")
+					(unit 1)
+				)
+				(path "/e63e39d7-6ac0-4ffd-8aa3-1841a4541b55/90e1f016-3c60-4383-aa8d-def9977ac47b/be7e522f-a717-4004-b2b4-d0582d753e6f"
+					(reference "#PWR0134")
 					(unit 1)
 				)
@@
 		(on_board yes)
 		(dnp no)
-		(property "Reference" "#PWR0100"
+		(property "Reference" "#PWR0115"
 			(at 71.12 24.13 0)
 			(effects
@@
 			(project ""
 				(path "/e63e39d7-6ac0-4ffd-8aa3-1841a4541b55/90e1f016-3c60-4383-aa8d-def9977ac47b/080e9e7b-a3e6-4d7b-a91a-d4d1bce9fcbf"
-					(reference "#PWR0100")
-					(unit 1)
-				)
-				(path "/e63e39d7-6ac0-4ffd-8aa3-1841a4541b55/90e1f016-3c60-4383-aa8d-def9977ac47b/0e21d398-15c6-48fd-a9a5-1cc9fd257aa3"
-					(reference "#PWR0110")
-					(unit 1)
-				)
-				(path "/e63e39d7-6ac0-4ffd-8aa3-1841a4541b55/90e1f016-3c60-4383-aa8d-def9977ac47b/763856e2-a839-4490-96d3-1a5f6bf03d10"
-					(reference "#PWR0105")
-					(unit 1)
-				)
-				(path "/e63e39d7-6ac0-4ffd-8aa3-1841a4541b55/90e1f016-3c60-4383-aa8d-def9977ac47b/be7e522f-a717-4004-b2b4-d0582d753e6f"
 					(reference "#PWR0115")
+					(unit 1)
+				)
+				(path "/e63e39d7-6ac0-4ffd-8aa3-1841a4541b55/90e1f016-3c60-4383-aa8d-def9977ac47b/0e21d398-15c6-48fd-a9a5-1cc9fd257aa3"
+					(reference "#PWR0125")
+					(unit 1)
+				)
+				(path "/e63e39d7-6ac0-4ffd-8aa3-1841a4541b55/90e1f016-3c60-4383-aa8d-def9977ac47b/763856e2-a839-4490-96d3-1a5f6bf03d10"
+					(reference "#PWR0120")
+					(unit 1)
+				)
+				(path "/e63e39d7-6ac0-4ffd-8aa3-1841a4541b55/90e1f016-3c60-4383-aa8d-def9977ac47b/be7e522f-a717-4004-b2b4-d0582d753e6f"
+					(reference "#PWR0130")
 					(unit 1)
 				)
@@
 		(on_board yes)
 		(dnp no)
-		(property "Reference" "#PWR0102"
+		(property "Reference" "#PWR0117"
 			(at 71.12 100.33 0)
 			(effects
@@
 			(project "fnx51"
 				(path "/e63e39d7-6ac0-4ffd-8aa3-1841a4541b55/90e1f016-3c60-4383-aa8d-def9977ac47b/080e9e7b-a3e6-4d7b-a91a-d4d1bce9fcbf"
-					(reference "#PWR0102")
-					(unit 1)
-				)
-				(path "/e63e39d7-6ac0-4ffd-8aa3-1841a4541b55/90e1f016-3c60-4383-aa8d-def9977ac47b/0e21d398-15c6-48fd-a9a5-1cc9fd257aa3"
-					(reference "#PWR0112")
-					(unit 1)
-				)
-				(path "/e63e39d7-6ac0-4ffd-8aa3-1841a4541b55/90e1f016-3c60-4383-aa8d-def9977ac47b/763856e2-a839-4490-96d3-1a5f6bf03d10"
-					(reference "#PWR0107")
-					(unit 1)
-				)
-				(path "/e63e39d7-6ac0-4ffd-8aa3-1841a4541b55/90e1f016-3c60-4383-aa8d-def9977ac47b/be7e522f-a717-4004-b2b4-d0582d753e6f"
 					(reference "#PWR0117")
+					(unit 1)
+				)
+				(path "/e63e39d7-6ac0-4ffd-8aa3-1841a4541b55/90e1f016-3c60-4383-aa8d-def9977ac47b/0e21d398-15c6-48fd-a9a5-1cc9fd257aa3"
+					(reference "#PWR0127")
+					(unit 1)
+				)
+				(path "/e63e39d7-6ac0-4ffd-8aa3-1841a4541b55/90e1f016-3c60-4383-aa8d-def9977ac47b/763856e2-a839-4490-96d3-1a5f6bf03d10"
+					(reference "#PWR0122")
+					(unit 1)
+				)
+				(path "/e63e39d7-6ac0-4ffd-8aa3-1841a4541b55/90e1f016-3c60-4383-aa8d-def9977ac47b/be7e522f-a717-4004-b2b4-d0582d753e6f"
+					(reference "#PWR0132")
 					(unit 1)
 				)
@@
 		(dnp no)
 		(fields_autoplaced yes)
-		(property "Reference" "U24"
+		(property "Reference" "U15"
 			(at 93.98 55.8799 90)
 			(effects
@@
 			(project ""
 				(path "/e63e39d7-6ac0-4ffd-8aa3-1841a4541b55/90e1f016-3c60-4383-aa8d-def9977ac47b/080e9e7b-a3e6-4d7b-a91a-d4d1bce9fcbf"
-					(reference "U24")
-					(unit 1)
-				)
-				(path "/e63e39d7-6ac0-4ffd-8aa3-1841a4541b55/90e1f016-3c60-4383-aa8d-def9977ac47b/0e21d398-15c6-48fd-a9a5-1cc9fd257aa3"
-					(reference "U24")
+					(reference "U15")
+					(unit 1)
+				)
+				(path "/e63e39d7-6ac0-4ffd-8aa3-1841a4541b55/90e1f016-3c60-4383-aa8d-def9977ac47b/0e21d398-15c6-48fd-a9a5-1cc9fd257aa3"
+					(reference "U15")
 					(unit 3)
 				)
 				(path "/e63e39d7-6ac0-4ffd-8aa3-1841a4541b55/90e1f016-3c60-4383-aa8d-def9977ac47b/763856e2-a839-4490-96d3-1a5f6bf03d10"
-					(reference "U24")
+					(reference "U15")
 					(unit 2)
 				)
 				(path "/e63e39d7-6ac0-4ffd-8aa3-1841a4541b55/90e1f016-3c60-4383-aa8d-def9977ac47b/be7e522f-a717-4004-b2b4-d0582d753e6f"
-					(reference "U24")
+					(reference "U15")
 					(unit 4)
 				)

Commit message: WIP PCB (add bypass caps, minor fixes)
Parts:
- added C30, C31: 100nF, symbol Device:C_Small
- renumbered U15 to U11, U25 to U17, U23 to U25, U24 to U26
Connections:
- net +5V: now also C30.2, C31.2
- net GND: now also C30.1, C31.1
Other:
- moved on the sheet: U11A
