File: pcb/filter.kicad_sch (KiCad schematic)
At the start: 0 parts

Commit message: WIP PCB
Parts:
- added C? (x5): 1nF 1%, symbol Device:C
- added C? (x2): 2.2nF 1%, symbol Device:C
- added C?: 3.3nF 1%, symbol Device:C
- added C? (x2): 0.1µF, symbol Device:C_Small
- added C? (x2): 10µF, symbol Device:C_Polarized_Small
- added C?: 18nF 1%, symbol Device:C
- added D? (x6): D_Filled, symbol Device:D_Filled
- added R? (x8): 33kΩ, symbol Device:R
- added R? (x2): 330kΩ, symbol Device:R
- added R?: 120kΩ, symbol Device:R
- added R?: 30kΩ, symbol Device:R
- added R?: 56kΩ, symbol Device:R
- added R?: 10kΩ, symbol Device:R
- added R? (x2): 2kΩ, symbol Device:R
- added R?: 130kΩ, symbol Device:R
- added TP? (x3): TestPoint_Probe, symbol Connector:TestPoint_Probe
- added U? (x3): TL072, symbol Amplifier_Operational:TL072
- added U? (x5): TL074, symbol Amplifier_Operational:TL074
Connections:
- new net: R?.1, R?.1, U?.6 (-), U?.7
- new net: R?.2, R?.2, U?.12 (+)
- new net: R?.1, R?.2, R?.2, U?.9 (-)
- new net: D?.1 (K), R?.2, R?.2
- new net: C?.1, R?.1, R?.2 (x2)
- new net: C?.1, R?.2, U?.3 (+)
- new net: C?.2, D?.1 (K), D?.2 (A) (x5)
- new net: C?.2, R?.1, TP?.1, U?.1, U?.2 (-)
- new net: C?.1, R?.2, U?.5 (+)
- new net: C?.2, R?.1, TP?.1, U?.6 (-), U?.7
- new net: R?.1, R?.2, U?.5 (+)
- new net: R?.1, R?.2, U?.13 (-)
- new net: R?.1, U?.14
- new net: C?.1, C?.1
- new net: R?.1, U?.8
- new net: R?.1, R?.2, U?.3 (+)
- new net: R?.1, R?.1, U?.1, U?.2 (-)
- new net: D?.2 (A), R?.2, R?.2
- new net +9VA: C?.1, C?.1, U?.4 (V+), U?.4 (V-)
- new net -9VA: C?.2, C?.2, U?.11 (V-), U?.8 (V+)
- new net GNDA: C?.1, C?.1, C?.1, C?.1, C?.1, C?.2, C?.2, C?.2, C?.2, R?.1, R?.2, R?.2, U?.10 (+)
- new net IN: R?.1
- new net PWM: R?.1, TP?.1
Other:
- note added: "Bulk Decoupling"
- note added: "PWM to CV"

Commit message: WIP PCB
Changed lines of the file:
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@@
 		)
 	)
+	(hierarchical_label "RESON0"
+		(shape input)
+		(at 96.52 88.9 0)
+		(effects
+			(font
+				(size 1.27 1.27)
+			)
+			(justify left)
+		)
+	)
+	(hierarchical_label "Z0"
+		(shape bidirectional)
+		(at 215.9 87.63 0)
+		(effects
+			(font
+				(size 1.27 1.27)
+			)
+			(justify left)
+		)
+	)
 	(hierarchical_label "IN"
 		(shape input)
@@
 		)
 	)
+	(hierarchical_label "Z1"
+		(shape bidirectional)
+		(at 217.17 96.52 0)
+		(effects
+			(font
+				(size 1.27 1.27)
+			)
+			(justify left)
+		)
+	)
+	(hierarchical_label "SELECT"
+		(shape input)
+		(at 96.52 99.06 0)
+		(effects
+			(font
+				(size 1.27 1.27)
+			)
+			(justify left)
+		)
+	)
+	(hierarchical_label "OUT"
+		(shape output)
+		(at 318.77 106.68 0)
+		(effects
+			(font
+				(size 1.27 1.27)
+			)
+			(justify left)
+		)
+	)
+	(hierarchical_label "RESON1"
+		(shape input)
+		(at 96.52 92.71 0)
+		(effects
+			(font
+				(size 1.27 1.27)
+			)
+			(justify left)
+		)
+	)
+	(hierarchical_label "Z"
+		(shape bidirectional)
+		(at 236.22 92.71 0)
+		(effects
+			(font
+				(size 1.27 1.27)
+			)
+			(justify left)
+		)
+	)
 	(symbol
 		(lib_id "Device:R")
@@
 		(dnp no)
 		(fields_autoplaced yes)
-		(property "Reference" "#PWR017"
+		(property "Reference" "#PWR?"
 			(at 257.81 173.99 0)
 			(effects
@@
 			(project "fnx51"
 				(path "/e63e39d7-6ac0-4ffd-8aa3-1841a4541b55/e4316b5d-360e-48fb-bbae-940258b1c798/43d9a0d9-77bd-4146-99af-cf6927920271"
-					(reference "#PWR017")
+					(reference "#PWR?")
 					(unit 1)
 				)
@@
 		(dnp no)
 		(fields_autoplaced yes)
-		(property "Reference" "#PWR05"
+		(property "Reference" "#PWR?"
 			(at 90.17 160.02 0)
 			(effects
@@
 			(project "fnx51"
 				(path "/e63e39d7-6ac0-4ffd-8aa3-1841a4541b55/e4316b5d-360e-48fb-bbae-940258b1c798/43d9a0d9-77bd-4146-99af-cf6927920271"
-					(reference "#PWR05")
+					(reference "#PWR?")
 					(unit 1)
 				)
@@
 		(on_board yes)
 		(dnp no)
-		(property "Reference" "#PWR016"
+		(property "Reference" "#PWR?"
 			(at 162.56 149.86 0)
 			(effects
@@
 			(project "fnx51"
 				(path "/e63e39d7-6ac0-4ffd-8aa3-1841a4541b55/e4316b5d-360e-48fb-bbae-940258b1c798/43d9a0d9-77bd-4146-99af-cf6927920271"
-					(reference "#PWR016")
+					(reference "#PWR?")
 					(unit 1)
 				)
@@
 		(dnp no)
 		(fields_autoplaced yes)
-		(property "Reference" "#PWR014"
+		(property "Reference" "#PWR?"
 			(at 203.2 171.45 0)
 			(effects
@@
 			(project "fnx51"
 				(path "/e63e39d7-6ac0-4ffd-8aa3-1841a4541b55/e4316b5d-360e-48fb-bbae-940258b1c798/43d9a0d9-77bd-4146-99af-cf6927920271"
-					(reference "#PWR014")
+					(reference "#PWR?")
 					(unit 1)
 				)
@@
 		(dnp no)
 		(fields_autoplaced yes)
-		(property "Reference" "#PWR04"
+		(property "Reference" "#PWR?"
 			(at 86.36 170.18 0)
 			(effects
@@
 			(project "fnx51"
 				(path "/e63e39d7-6ac0-4ffd-8aa3-1841a4541b55/e4316b5d-360e-48fb-bbae-940258b1c798/43d9a0d9-77bd-4146-99af-cf6927920271"
-					(reference "#PWR04")
+					(reference "#PWR?")
 					(unit 1)
 				)
@@
 		(dnp no)
 		(fields_autoplaced yes)
-		(property "Reference" "#PWR011"
+		(property "Reference" "#PWR?"
 			(at 143.51 241.3 0)
 			(effects
@@
 			(project "fnx51"
 				(path "/e63e39d7-6ac0-4ffd-8aa3-1841a4541b55/e4316b5d-360e-48fb-bbae-940258b1c798/43d9a0d9-77bd-4146-99af-cf6927920271"
-					(reference "#PWR011")
+					(reference "#PWR?")
 					(unit 1)
 				)
@@
 		(dnp no)
 		(fields_autoplaced yes)
-		(property "Reference" "#PWR010"
+		(property "Reference" "#PWR?"
 			(at 113.03 232.41 0)
 			(effects
@@
 			(project "fnx51"
 				(path "/e63e39d7-6ac0-4ffd-8aa3-1841a4541b55/e4316b5d-360e-48fb-bbae-940258b1c798/43d9a0d9-77bd-4146-99af-cf6927920271"
-					(reference "#PWR010")
+					(reference "#PWR?")
 					(unit 1)
 				)
@@
 		(on_board yes)
 		(dnp no)
-		(property "Reference" "#PWR02"
+		(property "Reference" "#PWR?"
 			(at 77.47 212.09 0)
 			(effects
@@
 			(project "fnx51"
 				(path "/e63e39d7-6ac0-4ffd-8aa3-1841a4541b55/e4316b5d-360e-48fb-bbae-940258b1c798/43d9a0d9-77bd-4146-99af-cf6927920271"
-					(reference "#PWR02")
+					(reference "#PWR?")
 					(unit 1)
 				)
@@
 		(on_board yes)
 		(dnp no)
-		(property "Reference" "#PWR08"
+		(property "Reference" "#PWR?"
 			(at 96.52 237.49 0)
 			(effects
@@
 			(project "fnx51"
 				(path "/e63e39d7-6ac0-4ffd-8aa3-1841a4541b55/e4316b5d-360e-48fb-bbae-940258b1c798/43d9a0d9-77bd-4146-99af-cf6927920271"
-					(reference "#PWR08")
+					(reference "#PWR?")
 					(unit 1)
 				)
@@
 		(dnp no)
 		(fields_autoplaced yes)
-		(property "Reference" "#PWR012"
+		(property "Reference" "#PWR?"
 			(at 203.2 236.22 0)
 			(effects
@@
 			(project "fnx51"
 				(path "/e63e39d7-6ac0-4ffd-8aa3-1841a4541b55/e4316b5d-360e-48fb-bbae-940258b1c798/43d9a0d9-77bd-4146-99af-cf6927920271"
-					(reference "#PWR012")
+					(reference "#PWR?")
 					(unit 1)
 				)
@@
 		(dnp no)
 		(fields_autoplaced yes)
-		(property "Reference" "#PWR06"
+		(property "Reference" "#PWR?"
 			(at 90.17 165.1 0)
 			(effects
@@
 			(project "fnx51"
 				(path "/e63e39d7-6ac0-4ffd-8aa3-1841a4541b55/e4316b5d-360e-48fb-bbae-940258b1c798/43d9a0d9-77bd-4146-99af-cf6927920271"
-					(reference "#PWR06")
+					(reference "#PWR?")
 					(unit 1)
 				)
@@
 		(on_board yes)
 		(dnp no)
-		(property "Reference" "#PWR03"
+		(property "Reference" "#PWR?"
 			(at 77.47 219.71 0)
 			(effects
@@
 			(project "fnx51"
 				(path "/e63e39d7-6ac0-4ffd-8aa3-1841a4541b55/e4316b5d-360e-48fb-bbae-940258b1c798/43d9a0d9-77bd-4146-99af-cf6927920271"
-					(reference "#PWR03")
+					(reference "#PWR?")
 					(unit 1)
 				)
@@
 		(on_board yes)
 		(dnp no)
-		(property "Reference" "#PWR015"
+		(property "Reference" "#PWR?"
 			(at 162.56 142.24 0)
 			(effects
@@
 			(project "fnx51"
 				(path "/e63e39d7-6ac0-4ffd-8aa3-1841a4541b55/e4316b5d-360e-48fb-bbae-940258b1c798/43d9a0d9-77bd-4146-99af-cf6927920271"
-					(reference "#PWR015")
+					(reference "#PWR?")
 					(unit 1)
 				)
@@
 		(dnp no)
 		(fields_autoplaced yes)
-		(property "Reference" "#PWR01"
+		(property "Reference" "#PWR?"
 			(at 66.04 232.41 0)
 			(effects
@@
 			(project "fnx51"
 				(path "/e63e39d7-6ac0-4ffd-8aa3-1841a4541b55/e4316b5d-360e-48fb-bbae-940258b1c798/43d9a0d9-77bd-4146-99af-cf6927920271"
-					(reference "#PWR01")
+					(reference "#PWR?")
 					(unit 1)
 				)
@@
 		(dnp no)
 		(fields_autoplaced yes)
-		(property "Reference" "#PWR013"
+		(property "Reference" "#PWR?"
 			(at 143.51 165.1 0)
 			(effects
@@
 			(project "fnx51"
 				(path "/e63e39d7-6ac0-4ffd-8aa3-1841a4541b55/e4316b5d-360e-48fb-bbae-940258b1c798/43d9a0d9-77bd-4146-99af-cf6927920271"
-					(reference "#PWR013")
+					(reference "#PWR?")
 					(unit 1)
 				)
@@
 		(on_board yes)
 		(dnp no)
-		(property "Reference" "#PWR09"
+		(property "Reference" "#PWR?"
 			(at 96.52 242.57 0)
 			(effects
@@
 			(project "fnx51"
 				(path "/e63e39d7-6ac0-4ffd-8aa3-1841a4541b55/e4316b5d-360e-48fb-bbae-940258b1c798/43d9a0d9-77bd-4146-99af-cf6927920271"
-					(reference "#PWR09")
+					(reference "#PWR?")
 					(unit 1)
 				)
@@
 		(dnp no)
 		(fields_autoplaced yes)
-		(property "Reference" "#PWR07"
+		(property "Reference" "#PWR?"
 			(at 92.71 247.65 0)
 			(effects
@@
 			(project "fnx51"
 				(path "/e63e39d7-6ac0-4ffd-8aa3-1841a4541b55/e4316b5d-360e-48fb-bbae-940258b1c798/43d9a0d9-77bd-4146-99af-cf6927920271"
-					(reference "#PWR07")
+					(reference "#PWR?")
 					(unit 1)
 				)

Commit message: wip schematic
Parts:
- added U?: 4053, symbol 4xxx:4053
Connections:
- net RESON0: now also U?.11 (A)
- net RESON1: now also U?.10 (B)
- net SELECT: now also U?.9 (C)
- net Z: now also U?.4 (Z)
- net Z0: now also U?.5 (Z0)
- net Z1: now also U?.3 (Z1)
Changed lines of the file:
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@@
 	(hierarchical_label "RESON0"
 		(shape input)
-		(at 96.52 88.9 0)
+		(at 213.36 100.33 180)
 		(effects
 			(font
 				(size 1.27 1.27)
 			)
-			(justify left)
+			(justify right)
 		)
 	)
 	(hierarchical_label "Z0"
 		(shape bidirectional)
-		(at 215.9 87.63 0)
+		(at 213.36 90.17 180)
 		(effects
 			(font
 				(size 1.27 1.27)
 			)
-			(justify left)
+			(justify right)
 		)
 	)
@@
 	(hierarchical_label "Z1"
 		(shape bidirectional)
-		(at 217.17 96.52 0)
+		(at 213.36 92.71 180)
 		(effects
 			(font
 				(size 1.27 1.27)
 			)
-			(justify left)
+			(justify right)
 		)
 	)
 	(hierarchical_label "SELECT"
 		(shape input)
-		(at 96.52 99.06 0)
+		(at 213.36 105.41 180)
 		(effects
 			(font
 				(size 1.27 1.27)
 			)
-			(justify left)
+			(justify right)
 		)
 	)
 	(hierarchical_label "OUT"
 		(shape output)
-		(at 318.77 106.68 0)
+		(at 326.39 165.1 0)
 		(effects
 			(font
@@
 	(hierarchical_label "RESON1"
 		(shape input)
-		(at 96.52 92.71 0)
+		(at 213.36 102.87 180)
 		(effects
 			(font
 				(size 1.27 1.27)
 			)
-			(justify left)
+			(justify right)
 		)
 	)
 	(hierarchical_label "Z"
 		(shape bidirectional)
-		(at 236.22 92.71 0)
+		(at 238.76 90.17 0)
 		(effects
 			(font
@@
 		)
 		(instances
+			(project ""
+				(path "/e63e39d7-6ac0-4ffd-8aa3-1841a4541b55/e4316b5d-360e-48fb-bbae-940258b1c798/43d9a0d9-77bd-4146-99af-cf6927920271"
+					(reference "U?")
+					(unit 1)
+				)
+			)
+		)
+	)
+	(symbol
+		(lib_id "4xxx:4053")
+		(at 226.06 90.17 0)
+		(unit 1)
+		(exclude_from_sim no)
+		(in_bom yes)
+		(on_board yes)
+		(dnp no)
+		(fields_autoplaced yes)
+		(property "Reference" "U?"
+			(at 228.2541 67.31 0)
+			(effects
+				(font
+					(size 1.27 1.27)
+				)
+				(justify left)
+			)
+		)
+		(property "Value" "4053"
+			(at 228.2541 69.85 0)
+			(effects
+				(font
+					(size 1.27 1.27)
+				)
+				(justify left)
+			)
+		)
+		(property "Footprint" ""
+			(at 226.06 90.17 0)
+			(effects
+				(font
+					(size 1.27 1.27)
+				)
+				(hide yes)
+			)
+		)
+		(property "Datasheet" "http://www.intersil.com/content/dam/Intersil/documents/cd40/cd4051bms-52bms-53bms.pdf"
+			(at 226.06 90.17 0)
+			(effects
+				(font
+					(size 1.27 1.27)
+				)
+				(hide yes)
+			)
+		)
+		(property "Description" "Triple analog Multiplexer 2 to 1 line"
+			(at 226.06 90.17 0)
+			(effects
+				(font
+					(size 1.27 1.27)
+				)
+				(hide yes)
+			)
+		)
+		(pin "4"
+		)
+		(pin "12"
+		)
+		(pin "10"
+		)
+		(pin "8"
+		)
+		(pin "9"
+		)
+		(pin "5"
+		)
+		(pin "16"
+		)
+		(pin "11"
+		)
+		(pin "15"
+		)
+		(pin "3"
+		)
+		(pin "13"
+		)
+		(pin "2"
+		)
+		(pin "6"
+		)
+		(pin "7"
+		)
+		(pin "14"
+		)
+		(pin "1"
+		)
+		(instances

Commit message: PCB: add reset circuit, xtal
Parts:
- gave numbers to parts that had none: 42

Commit message: WIP schematic
Parts:
- renumbered C67 to C71, C68 to C72, C69 to C73, C70 to C74, C71 to C75, C72 to C76, C73 to C77, C74 to C78, C75 to C79, C76 to C80, C77 to C81, C78 to C82, C79 to C83, D9 to D10, D10 to D11, D11 to D12, D6 to D7, D7 to D8, D8 to D9, R103 to R110, R104 to R111, R105 to R112, R106 to R113, R107 to R114, R108 to R115, R109 to R116, R110 to R117, R111 to R118, R112 to R119, R113 to R120, R114 to R121, R115 to R122, R116 to R123, R117 to R124, R118 to R125, R119 to R126, U80 to U81, U81 to U82, U82 to U83

Commit message: WIP schematic
Parts:
- added C90, C96: 1µF, symbol Device:C
- added D15, D16: 1N4148, symbol Device:D_Filled
- added R130, R152: 200kΩ, symbol Device:R
- added R144: 43kΩ, symbol Device:R
- added R145: 8.2kΩ, symbol Device:R
- added R146, R148, R149: 20kΩ, symbol Device:R
- added R147: 10kΩ, symbol Device:R
- added R150: 1kΩ, symbol Device:R
- added R151: 47kΩ, symbol Device:R
- added TP49, TP50, TP51, TP52: TestPoint_Probe, symbol Connector:TestPoint_Probe
- added U66: TL074, symbol Amplifier_Operational:TL074
- D10: renamed from D8; value D_Filled -> 1N4148
- D11: renamed from D9; value D_Filled -> 1N4148
- D12: renamed from D10; value D_Filled -> 1N4148
- D13: renamed from D11; value D_Filled -> 1N4148
- D14: renamed from D12; value D_Filled -> 1N4148
- D9: renamed from D7; value D_Filled -> 1N4148
- R132: renamed from R115; value 330kΩ -> 330Ω
- renumbered C71 to C82, C72 to C83, C73 to C84, C74 to C85, C75 to C86, C76 to C87, C77 to C88, C78 to C89, C79 to C91, C80 to C92, C81 to C93, C82 to C94, C83 to C95, R110 to R126, R111 to R127, R112 to R128, R113 to R129, R114 to R131, R116 to R133, R117 to R134, R118 to R135, R119 to R136, R120 to R137, R121 to R138, R122 to R139, R123 to R140, R124 to R141, R125 to R142, R126 to R143, TP44 to TP46, TP45 to TP47, TP46 to TP48, U81 to U82, U82 to U83, U83 to U84
Connections:
- net +9VA: now also U84.16 (VDD), U66.4 (V+)
- net -9VA: now also U84.7 (VEE), U66.11 (V-)
- net GNDA: now also U84.12 (X0), U84.2 (Y0), U84.8 (VSS), R130.2, R145.1, R149.1, R152.2, U66.12 (+)
- net IN: now also C90.1; no longer R131.1
- net OUT: now also C96.1
- net RESON0: now also U84.10 (B); no longer U84.11 (A)
- net RESON1: now also U84.11 (A); no longer U84.10 (B)
- net at D14.1 (K), R141.2, R143.2: now also TP51.1
- net at C93.2, D11.1 (K), D12.2 (A): now also U66.3 (+)
- net at C91.1, C95.1: now also D15.2 (A), D16.1 (K), R144.2, U66.7
- net at R135.1, R137.1, U83.1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: now also TP49.1
- net at D9.2 (A), R140.2, R142.2: now also TP50.1
- net at U84.1 (Y1): now also U84.13 (X1), R150.2, TP52.1, U66.1, U66.2 (-)
- net at U84.14 (X): now also R146.1
- net at U84.15 (Y): now also R148.1
- new net: D15.1 (K), D16.2 (A), R144.1, R145.2, U66.6 (-)
- new net: R147.1, R148.2, R149.2
- new net: R146.2, R147.2, U66.5 (+)
- new net: C90.2, R130.1, R131.1
- new net: C96.2, R151.1, R152.1, U66.14
- new net: R150.1, R151.2, U66.13 (-)
Other:
- moved on the sheet: U84

Commit message: WIP schematic
Parts:
- renumbered C95 to C100, C96 to C101, C82 to C87, C83 to C88, C84 to C89, C85 to C90, C86 to C91, C87 to C92, C88 to C93, C89 to C94, C90 to C95, C91 to C96, C92 to C97, C93 to C98, C94 to C99
Connections:
- net GNDA: now also U84.6 (Inh)

Commit message: WIP PCB (add bypass caps, minor fixes)
Parts:
- renumbered C87 to C137, C88 to C138, C89 to C139, C90 to C140, C91 to C141, C92 to C142, C93 to C143, C94 to C144, C95 to C145, C96 to C146, C97 to C147, C98 to C148, C99 to C149, C100 to C150, C101 to C151, R126 to R129, R127 to R130, R128 to R131, R129 to R132, R130 to R133, R131 to R134, R132 to R135, R133 to R136, R134 to R137, R135 to R138, R136 to R139, R137 to R140, R138 to R141, R139 to R142, R140 to R143, R141 to R144, R142 to R145, R143 to R146, R144 to R147, R145 to R148, R146 to R149, R147 to R150, R148 to R151, R149 to R152, R150 to R153, R151 to R154, R152 to R155
