File: pcb/filter.kicad_sch (KiCad schematic)
At the start: 61 parts, among them U66 TL074, U82 TL072, U83 TL074, U84 4053

Commit message: update to kicad 10 and fix vertical video timing
Parts:
- renumbered R129 to R130, R130 to R131, R131 to R132, R132 to R133, R133 to R134, R134 to R135, R135 to R136, R136 to R137, R137 to R138, R138 to R139, R139 to R140, R140 to R141, R141 to R142, R142 to R143, R143 to R144, R144 to R145, R145 to R146, R146 to R147, R147 to R148, R148 to R149, R149 to R150, R150 to R151, R151 to R152, R152 to R153, R153 to R154, R154 to R155, R155 to R156
