File: pcb/voice.kicad_sch (KiCad schematic)
At the start: 45 parts, among them Q2 BC547, Q4 BC547, Q6 BC547, U52 TL074, U55 TL074, U56 TL072, U57 TL074

Commit message: WIP schematic
Parts:
- added R26, R27: 56kΩ, symbol Device:R
- added TP14: TestPoint_Probe, symbol Connector:TestPoint_Probe
- renumbered C21 to C25, C22 to C26, C19 to C27, C6 to C28, C23 to C29, C10 to C30, C11 to C31, C12 to C32, C13 to C33, C14 to C34, C15 to C35, C30 to C36, C17 to C37, C18 to C38, Q4 to Q7, Q2 to Q8, Q6 to Q9, R1 to R35, R2 to R36, R3 to R37, R4 to R38, R5 to R39, R6 to R40, R7 to R41, R8 to R42, R9 to R43, R10 to R46, R11 to R47, R12 to R48, R13 to R49, R30 to R50, R31 to R51, R32 to R52, TP9 to TP17, TP2 to TP18, TP3 to TP19, TP4 to TP20, TP5 to TP21, TP6 to TP22, TP7 to TP24, TP8 to TP25, U56 to U65, U55 to U66, U52 to U66, U57 to U67
Connections:
- net GNDA: now also U66.10 (+), U66.3 (+), U66.5 (+); no longer U65.3 (+), U65.5 (+), U66.12 (+)
- net PWM: now also R35.1, TP17.1; no longer U66.3 (+)
- net at Q8.1 (C), R43.1: now also U66.9 (-); no longer U65.6 (-)
- net at C33.1, Q7.1 (C), R41.2: now also U66.6 (-); no longer U65.2 (-)
- net at Q7.2 (B), R40.2, TP20.1: now also U66.1; no longer U66.14
- net at R39.2, R40.1: now also U66.2 (-); no longer U66.13 (-)
- net at C32.1, R38.2: now also U65.5 (+); no longer U66.10 (+)
- net at C25.2, R37.1, TP18.1: now also U65.1, U65.2 (-); no longer U66.6 (-), U66.7
- net at C33.2, R42.2, TP21.1: now also U66.7; no longer U65.1
- net at C31.2, R39.1, TP19.1: now also U65.6 (-), U65.7; no longer U66.8, U66.9 (-)
- net at C26.1, R36.2: now also U65.3 (+); no longer U66.5 (+)
- net +12V renamed +9VA
- net -12V renamed -9VA
- new net: R26.1, R43.2, TP22.1, U66.8
- new net: R46.1, R47.1, TP14.1, U66.13 (-), U66.14
- new net: R26.2, R27.1, U66.12 (+)
- new net FM/OCTAVE: R27.2
Other:
- note added: "FM"
- moved on the sheet: C25, C26, C29, C30, C31, C32, C33, C34, C35, C36, C37, C38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

Commit message: WIP PCB
Parts:
- renumbered C38 to C?, C28 to C?, C34 to C?, C32 to C?, C30 to C?, C27 to C?, C31 to C?, C37 to C?, C25 to C?, C36 to C?, C33 to C?, C29 to C?, C26 to C?, C35 to C?, Q8 to Q?, Q7 to Q?, Q9 to Q?, R48 to R?, R49 to R?, R47 to R?, R27 to R?, R37 to R?, R36 to R?, R51 to R?, R26 to R?, R46 to R?, R50 to R?, R40 to R?, R52 to R?, R43 to R?, R42 to R?, R38 to R?, R41 to R?, R35 to R?, R39 to R?, TP22 to TP?, TP21 to TP?, TP20 to TP?, TP18 to TP?, TP17 to TP?, TP25 to TP?, TP19 to TP?, TP14 to TP?, TP24 to TP?, U65 to U?, U66 to U?, U67 to U?
Other:
- note added: "PVM to CV"
- note removed: "Low-Pass Filter"

Commit message: wip schematic
Other:
- note added: "PWM to CV"
- note removed: "PVM to CV"
Changed lines of the file:
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@@
 		)
 	)
-	(text "PVM to CV"
+	(text "PWM to CV"
 		(exclude_from_sim no)
 		(at 30.48 116.84 0)

Commit message: PCB: add reset circuit, xtal
Parts:
- gave numbers to parts that had none: 47

Commit message: WIP schematic
Parts:
- renumbered C11 to C15, C12 to C16, C13 to C17, C14 to C18, C15 to C19, C16 to C20, C17 to C21, C18 to C22, C19 to C23, C20 to C24, C21 to C25, C22 to C26, C23 to C27, C24 to C28, Q8 to Q11, Q9 to Q12, Q10 to Q13, R31 to R38, R32 to R39, R33 to R40, R34 to R41, R35 to R42, R36 to R43, R37 to R44, R38 to R45, R39 to R46, R40 to R47, R41 to R48, R42 to R49, R43 to R50, R44 to R51, R45 to R52, R46 to R53, R47 to R54, R48 to R55, U68 to U69, U69 to U70, U70 to U71

Commit message: WIP schematic
Parts:
- renumbered C15 to C26, C16 to C27, C17 to C28, C18 to C29, C19 to C30, C20 to C31, C21 to C32, C22 to C33, C23 to C34, C24 to C35, C25 to C36, C26 to C37, C27 to C38, C28 to C39, Q11 to Q13, Q12 to Q14, Q13 to Q15, R38 to R54, R39 to R55, R40 to R56, R41 to R57, R42 to R58, R43 to R59, R44 to R60, R45 to R61, R46 to R62, R47 to R63, R48 to R64, R49 to R65, R50 to R66, R51 to R67, R52 to R68, R53 to R69, R54 to R70, R55 to R71, TP8 to TP10, TP9 to TP11, TP10 to TP12, TP11 to TP13, TP12 to TP14, TP13 to TP15, TP14 to TP16, TP15 to TP17, TP16 to TP18, U69 to U70, U70 to U71, U71 to U72

Commit message: WIP schematic
Parts:
- renumbered C26 to C31, C27 to C32, C28 to C33, C29 to C34, C30 to C35, C31 to C36, C32 to C37, C33 to C38, C34 to C39, C35 to C40, C36 to C41, C37 to C42, C38 to C43, C39 to C44

Commit message: WIP PCB (add bypass caps, minor fixes)
Parts:
- renumbered C31 to C81, C32 to C82, C33 to C83, C34 to C84, C35 to C85, C36 to C86, C37 to C87, C38 to C88, C39 to C89, C40 to C90, C41 to C91, C42 to C92, C43 to C93, C44 to C94, R54 to R57, R55 to R58, R56 to R59, R57 to R60, R58 to R61, R59 to R62, R60 to R63, R61 to R64, R62 to R65, R63 to R66, R64 to R67, R65 to R68, R66 to R69, R67 to R70, R68 to R71, R69 to R72, R70 to R73, R71 to R74
