File: pcb/voice.kicad_sch (KiCad schematic)
At the start: 47 parts, among them Q13 BC547, Q14 BC547, Q15 BC547, U70 TL072, U71 TL074, U72 TL074

Commit message: update to kicad 10 and fix vertical video timing
Parts:
- renumbered R57 to R58, R58 to R59, R59 to R60, R60 to R61, R61 to R62, R62 to R63, R63 to R64, R64 to R65, R65 to R66, R66 to R67, R67 to R68, R68 to R69, R69 to R70, R70 to R71, R71 to R72, R72 to R73, R73 to R74, R74 to R75
