File: pcb/vram8k.kicad_sch (KiCad schematic)
At the start: 1 part

Commit message: PCB: add reset circuit, xtal
Parts:
- gave numbers to parts that had none: 1
Connections:
- no-connect marks 3 -> 2
Changed lines of the file:
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@@
 (kicad_sch
-	(version 20231120)
+	(version 20250114)
 	(generator "eeschema")
-	(generator_version "8.0")
+	(generator_version "9.0")
 	(paper "A5" portrait)
 	(junction
@@
 	(no_connect
 		(at 90.17 125.73)
-	)
-	(no_connect
-		(at 69.85 121.92)
 	)
 	(wire
@@
 		(dnp no)
 		(fields_autoplaced yes)
-		(property "Reference" "#PWR?"
+		(property "Reference" "#PWR0137"
 			(at 72.39 35.56 0)
 			(effects
@@
 			(project ""
 				(path "/e63e39d7-6ac0-4ffd-8aa3-1841a4541b55/90e1f016-3c60-4383-aa8d-def9977ac47b/2da79d81-44d3-45bf-87cb-e571d3f74d12"
-					(reference "#PWR?")
+					(reference "#PWR0137")
 					(unit 1)
 				)
 				(path "/e63e39d7-6ac0-4ffd-8aa3-1841a4541b55/90e1f016-3c60-4383-aa8d-def9977ac47b/49e585c5-db3a-4822-8d59-7a86ce4b7919"
-					(reference "#PWR?")
+					(reference "#PWR0146")
 					(unit 1)
 				)
 				(path "/e63e39d7-6ac0-4ffd-8aa3-1841a4541b55/90e1f016-3c60-4383-aa8d-def9977ac47b/bed087ff-bb84-4587-ab14-e44eb20e33e5"
-					(reference "#PWR?")
+					(reference "#PWR0164")
 					(unit 1)
 				)
 				(path "/e63e39d7-6ac0-4ffd-8aa3-1841a4541b55/90e1f016-3c60-4383-aa8d-def9977ac47b/cf6a9fb3-feb6-497a-b217-8cd4e80219cd"
-					(reference "#PWR?")
+					(reference "#PWR0155")
 					(unit 1)
 				)
@@
 		(on_board yes)
 		(dnp no)
-		(property "Reference" "#PWR?"
+		(property "Reference" "#PWR0133"
 			(at 53.34 50.8 0)
 			(effects
@@
 			(project ""
 				(path "/e63e39d7-6ac0-4ffd-8aa3-1841a4541b55/90e1f016-3c60-4383-aa8d-def9977ac47b/2da79d81-44d3-45bf-87cb-e571d3f74d12"
-					(reference "#PWR?")
+					(reference "#PWR0133")
 					(unit 1)
 				)
 				(path "/e63e39d7-6ac0-4ffd-8aa3-1841a4541b55/90e1f016-3c60-4383-aa8d-def9977ac47b/49e585c5-db3a-4822-8d59-7a86ce4b7919"
-					(reference "#PWR?")
+					(reference "#PWR0142")
 					(unit 1)
 				)
 				(path "/e63e39d7-6ac0-4ffd-8aa3-1841a4541b55/90e1f016-3c60-4383-aa8d-def9977ac47b/bed087ff-bb84-4587-ab14-e44eb20e33e5"
-					(reference "#PWR?")
+					(reference "#PWR0160")
 					(unit 1)
 				)
 				(path "/e63e39d7-6ac0-4ffd-8aa3-1841a4541b55/90e1f016-3c60-4383-aa8d-def9977ac47b/cf6a9fb3-feb6-497a-b217-8cd4e80219cd"
-					(reference "#PWR?")
+					(reference "#PWR0151")
 					(unit 1)
 				)
@@
 		(dnp no)
 		(fields_autoplaced yes)
-		(property "Reference" "#PWR?"
+		(property "Reference" "#PWR0138"
 			(at 91.44 52.07 0)
 			(effects
@@
 			(project "fnx51"
 				(path "/e63e39d7-6ac0-4ffd-8aa3-1841a4541b55/90e1f016-3c60-4383-aa8d-def9977ac47b/2da79d81-44d3-45bf-87cb-e571d3f74d12"
-					(reference "#PWR?")
+					(reference "#PWR0138")
 					(unit 1)
 				)
 				(path "/e63e39d7-6ac0-4ffd-8aa3-1841a4541b55/90e1f016-3c60-4383-aa8d-def9977ac47b/49e585c5-db3a-4822-8d59-7a86ce4b7919"
-					(reference "#PWR?")
+					(reference "#PWR0147")
 					(unit 1)
 				)
 				(path "/e63e39d7-6ac0-4ffd-8aa3-1841a4541b55/90e1f016-3c60-4383-aa8d-def9977ac47b/bed087ff-bb84-4587-ab14-e44eb20e33e5"
-					(reference "#PWR?")
+					(reference "#PWR0165")
 					(unit 1)
 				)
 				(path "/e63e39d7-6ac0-4ffd-8aa3-1841a4541b55/90e1f016-3c60-4383-aa8d-def9977ac47b/cf6a9fb3-feb6-497a-b217-8cd4e80219cd"
-					(reference "#PWR?")
+					(reference "#PWR0156")
 					(unit 1)
 				)
@@
 		(dnp no)
 		(fields_autoplaced yes)
-		(property "Reference" "U?"
+		(property "Reference" "U43"
 			(at 77.1241 36.83 0)
 			(effects
@@
 			(project ""
 				(path "/e63e39d7-6ac0-4ffd-8aa3-1841a4541b55/90e1f016-3c60-4383-aa8d-def9977ac47b/2da79d81-44d3-45bf-87cb-e571d3f74d12"
-					(reference "U?")
+					(reference "U43")
 					(unit 1)
 				)
 				(path "/e63e39d7-6ac0-4ffd-8aa3-1841a4541b55/90e1f016-3c60-4383-aa8d-def9977ac47b/49e585c5-db3a-4822-8d59-7a86ce4b7919"
-					(reference "U?")
+					(reference "U44")
 					(unit 1)
 				)
 				(path "/e63e39d7-6ac0-4ffd-8aa3-1841a4541b55/90e1f016-3c60-4383-aa8d-def9977ac47b/bed087ff-bb84-4587-ab14-e44eb20e33e5"
-					(reference "U?")
+					(reference "U46")
 					(unit 1)
 				)
 				(path "/e63e39d7-6ac0-4ffd-8aa3-1841a4541b55/90e1f016-3c60-4383-aa8d-def9977ac47b/cf6a9fb3-feb6-497a-b217-8cd4e80219cd"
-					(reference "U?")
+					(reference "U45")
 					(unit 1)
 				)
@@
 		(on_board yes)
 		(dnp no)
-		(property "Reference" "#PWR?"
+		(property "Reference" "#PWR0136"
 			(at 71.12 144.78 0)
 			(effects
@@
 			(project "fnx51"
 				(path "/e63e39d7-6ac0-4ffd-8aa3-1841a4541b55/90e1f016-3c60-4383-aa8d-def9977ac47b/2da79d81-44d3-45bf-87cb-e571d3f74d12"
-					(reference "#PWR?")
+					(reference "#PWR0136")
 					(unit 1)
 				)
 				(path "/e63e39d7-6ac0-4ffd-8aa3-1841a4541b55/90e1f016-3c60-4383-aa8d-def9977ac47b/49e585c5-db3a-4822-8d59-7a86ce4b7919"
-					(reference "#PWR?")
+					(reference "#PWR0145")
 					(unit 1)
 				)
 				(path "/e63e39d7-6ac0-4ffd-8aa3-1841a4541b55/90e1f016-3c60-4383-aa8d-def9977ac47b/bed087ff-bb84-4587-ab14-e44eb20e33e5"
-					(reference "#PWR?")
+					(reference "#PWR0163")
 					(unit 1)
 				)
 				(path "/e63e39d7-6ac0-4ffd-8aa3-1841a4541b55/90e1f016-3c60-4383-aa8d-def9977ac47b/cf6a9fb3-feb6-497a-b217-8cd4e80219cd"
-					(reference "#PWR?")
+					(reference "#PWR0154")
 					(unit 1)
 				)
@@
 		(on_board yes)
 		(dnp no)
-		(property "Reference" "#PWR?"
+		(property "Reference" "#PWR0135"
 			(at 53.34 127 0)
 			(effects
@@
 			(project "fnx51"
 				(path "/e63e39d7-6ac0-4ffd-8aa3-1841a4541b55/90e1f016-3c60-4383-aa8d-def9977ac47b/2da79d81-44d3-45bf-87cb-e571d3f74d12"
-					(reference "#PWR?")
+					(reference "#PWR0135")
 					(unit 1)
 				)
 				(path "/e63e39d7-6ac0-4ffd-8aa3-1841a4541b55/90e1f016-3c60-4383-aa8d-def9977ac47b/49e585c5-db3a-4822-8d59-7a86ce4b7919"
-					(reference "#PWR?")
+					(reference "#PWR0144")
 					(unit 1)
 				)
 				(path "/e63e39d7-6ac0-4ffd-8aa3-1841a4541b55/90e1f016-3c60-4383-aa8d-def9977ac47b/bed087ff-bb84-4587-ab14-e44eb20e33e5"
-					(reference "#PWR?")
+					(reference "#PWR0162")
 					(unit 1)
 				)
 				(path "/e63e39d7-6ac0-4ffd-8aa3-1841a4541b55/90e1f016-3c60-4383-aa8d-def9977ac47b/cf6a9fb3-feb6-497a-b217-8cd4e80219cd"
-					(reference "#PWR?")
+					(reference "#PWR0153")
 					(unit 1)
 				)
@@
 		(on_board yes)
 		(dnp no)
-		(property "Reference" "#PWR?"
+		(property "Reference" "#PWR0141"
 			(at 93.98 59.69 0)
 			(effects
@@
 			(project "fnx51"
 				(path "/e63e39d7-6ac0-4ffd-8aa3-1841a4541b55/90e1f016-3c60-4383-aa8d-def9977ac47b/2da79d81-44d3-45bf-87cb-e571d3f74d12"
-					(reference "#PWR?")
+					(reference "#PWR0141")
 					(unit 1)
 				)
 				(path "/e63e39d7-6ac0-4ffd-8aa3-1841a4541b55/90e1f016-3c60-4383-aa8d-def9977ac47b/49e585c5-db3a-4822-8d59-7a86ce4b7919"
-					(reference "#PWR?")
+					(reference "#PWR0150")
 					(unit 1)
 				)
 				(path "/e63e39d7-6ac0-4ffd-8aa3-1841a4541b55/90e1f016-3c60-4383-aa8d-def9977ac47b/bed087ff-bb84-4587-ab14-e44eb20e33e5"
-					(reference "#PWR?")
+					(reference "#PWR0168")
 					(unit 1)
 				)
 				(path "/e63e39d7-6ac0-4ffd-8aa3-1841a4541b55/90e1f016-3c60-4383-aa8d-def9977ac47b/cf6a9fb3-feb6-497a-b217-8cd4e80219cd"
-					(reference "#PWR?")
+					(reference "#PWR0159")
 					(unit 1)
 				)
@@
 		(on_board yes)
 		(dnp no)
-		(property "Reference" "#PWR?"
+		(property "Reference" "#PWR0140"
 			(at 91.44 127 0)
 			(effects
@@
 			(project "fnx51"
 				(path "/e63e39d7-6ac0-4ffd-8aa3-1841a4541b55/90e1f016-3c60-4383-aa8d-def9977ac47b/2da79d81-44d3-45bf-87cb-e571d3f74d12"
-					(reference "#PWR?")
+					(reference "#PWR0140")
 					(unit 1)
 				)
 				(path "/e63e39d7-6ac0-4ffd-8aa3-1841a4541b55/90e1f016-3c60-4383-aa8d-def9977ac47b/49e585c5-db3a-4822-8d59-7a86ce4b7919"
-					(reference "#PWR?")
+					(reference "#PWR0149")
 					(unit 1)
 				)
 				(path "/e63e39d7-6ac0-4ffd-8aa3-1841a4541b55/90e1f016-3c60-4383-aa8d-def9977ac47b/bed087ff-bb84-4587-ab14-e44eb20e33e5"
-					(reference "#PWR?")
+					(reference "#PWR0167")
 					(unit 1)
 				)
 				(path "/e63e39d7-6ac0-4ffd-8aa3-1841a4541b55/90e1f016-3c60-4383-aa8d-def9977ac47b/cf6a9fb3-feb6-497a-b217-8cd4e80219cd"
-					(reference "#PWR?")
+					(reference "#PWR0158")
 					(unit 1)
 				)
@@
 		(on_board yes)
 		(dnp no)
-		(property "Reference" "#PWR?"
+		(property "Reference" "#PWR0139"
 			(at 91.44 88.9 0)
 			(effects
@@
 			(project "fnx51"
 				(path "/e63e39d7-6ac0-4ffd-8aa3-1841a4541b55/90e1f016-3c60-4383-aa8d-def9977ac47b/2da79d81-44d3-45bf-87cb-e571d3f74d12"
-					(reference "#PWR?")
+					(reference "#PWR0139")
 					(unit 1)
 				)
 				(path "/e63e39d7-6ac0-4ffd-8aa3-1841a4541b55/90e1f016-3c60-4383-aa8d-def9977ac47b/49e585c5-db3a-4822-8d59-7a86ce4b7919"
-					(reference "#PWR?")
+					(reference "#PWR0148")
 					(unit 1)
 				)
 				(path "/e63e39d7-6ac0-4ffd-8aa3-1841a4541b55/90e1f016-3c60-4383-aa8d-def9977ac47b/bed087ff-bb84-4587-ab14-e44eb20e33e5"
-					(reference "#PWR?")
+					(reference "#PWR0166")
 					(unit 1)
 				)
 				(path "/e63e39d7-6ac0-4ffd-8aa3-1841a4541b55/90e1f016-3c60-4383-aa8d-def9977ac47b/cf6a9fb3-feb6-497a-b217-8cd4e80219cd"
-					(reference "#PWR?")
+					(reference "#PWR0157")
 					(unit 1)
 				)
@@
 		(on_board yes)
 		(dnp no)
-		(property "Reference" "#PWR?"
+		(property "Reference" "#PWR0134"
 			(at 53.34 86.36 0)
 			(effects
@@
 			(project "fnx51"
 				(path "/e63e39d7-6ac0-4ffd-8aa3-1841a4541b55/90e1f016-3c60-4383-aa8d-def9977ac47b/2da79d81-44d3-45bf-87cb-e571d3f74d12"
-					(reference "#PWR?")
+					(reference "#PWR0134")
 					(unit 1)
 				)
 				(path "/e63e39d7-6ac0-4ffd-8aa3-1841a4541b55/90e1f016-3c60-4383-aa8d-def9977ac47b/49e585c5-db3a-4822-8d59-7a86ce4b7919"
-					(reference "#PWR?")
+					(reference "#PWR0143")
 					(unit 1)
 				)
 				(path "/e63e39d7-6ac0-4ffd-8aa3-1841a4541b55/90e1f016-3c60-4383-aa8d-def9977ac47b/bed087ff-bb84-4587-ab14-e44eb20e33e5"
-					(reference "#PWR?")
+					(reference "#PWR0161")
 					(unit 1)
 				)
 				(path "/e63e39d7-6ac0-4ffd-8aa3-1841a4541b55/90e1f016-3c60-4383-aa8d-def9977ac47b/cf6a9fb3-feb6-497a-b217-8cd4e80219cd"
-					(reference "#PWR?")
-					(unit 1)
-				)
+					(reference "#PWR0152")
+					(unit 1)
+				)

Commit message: WIP schematic
Parts:
- renumbered U43 to U44

Commit message: WIP PCB (add bypass caps, minor fixes)
Parts:
- added C51: 100nF, symbol Device:C_Small
Connections:
- net +5V: now also C51.2
- net GND: now also C51.1
