File: pcb/audio.kicad_sch (KiCad schematic)
At the start: 76 parts, among them J9 Headphones, Q10 BC547, Q11 BC338, Q12 BC328, Q7 BC547, Q8 BC547, Q9 BC547, U58 74HC245, U59 4504, U60 4053, U61 4053, U62 4504, U63 4053, U64 TL072, U65 4053, U66 TL074, U67 LM7809_TO220, U68 LM7805_TO220, U69 LM7909_TO220

Commit message: update to kicad 10 and fix vertical video timing
Parts:
- renumbered R27 to R28, R28 to R29, R29 to R30, R30 to R31, R31 to R32, R32 to R33, R33 to R34, R34 to R35, R35 to R36, R36 to R37, R37 to R38, R38 to R39, R39 to R40, R40 to R41, R41 to R42, R42 to R43, R43 to R44, R44 to R45, R45 to R46, R46 to R47, R47 to R48, R48 to R49, R49 to R50, R50 to R51, R51 to R52, R52 to R53, R53 to R54, R54 to R55, R55 to R56, R56 to R57
