File: pcb/copro.kicad_sch (KiCad schematic)
At the start: 15 parts, among them U39 74HC02, U40 ATmega1284-P, U41 74HC245, U42 74HC245, U43 74HC245, Y2 20MHz

Commit message: update to kicad 10 and fix vertical video timing
Parts:
- renumbered R18 to R19, R19 to R20
Connections:
- net ~{VMAP}: no longer U43.19 (CE)
- net ~{VME}a: now also U43.19 (CE)
