File: pcb/ethernet.kicad_sch (KiCad schematic)
At the start: 22 parts, among them J7 Conn_01x01_Pin, J8 ARJM11A3-009-AB-ER2-T, U1 74HCT125, U57 ENC28J60x-SP, Y3 25MHz

Commit message: update to kicad 10 and fix vertical video timing
Parts:
- renumbered R20 to R21, R21 to R22, R22 to R23, R23 to R24, R24 to R25, R25 to R26, R26 to R27
Connections:
- net +3.3V: no longer J8.L1, J8.L4
- net GND: now also J8.L2, J8.L3, U1.1
- net SI: no longer U1.1
- net at R26.1: now also J8.L4; no longer J8.L3
- net at R27.1: now also J8.L1; no longer J8.L2
Other:
- moved on the sheet: R26, R27, U1A
