File: pcb/r2r.kicad_sch (KiCad schematic)
At the start: 8 parts

Commit message: update to kicad 10 and fix vertical video timing
Parts:
- renumbered R172 to R173, R173 to R174, R174 to R175, R175 to R176, R176 to R177, R177 to R178, R178 to R179, R179 to R180
