File: pcb/serial.kicad_sch (KiCad schematic)
At the start: 20 parts, among them J10 01x03, J11 01x03, J12 01x03, J13 01x03, J14 Mini-DIN-6, J15 Mini-DIN-6, J16 SHIELD, J17 DE9_Pins_MountingHoles, J18 01x09, J19 01x09, U94 MAX232

Commit message: update to kicad 10 and fix vertical video timing
Parts:
- renumbered R196 to R197, R197 to R198, R198 to R199, R199 to R200
