File: pcb/volume.kicad_sch (KiCad schematic)
At the start: 33 parts, among them U85 74LS573, U86 74LS573, U87 74LS573, U88 74LS573, U89 DAC0808_DIP, U90 DAC0808_DIP, U91 DAC0808_DIP, U92 DAC0808_DIP, U93 TL074

Commit message: update to kicad 10 and fix vertical video timing
Parts:
- renumbered R156 to R157, R157 to R158, R158 to R159, R159 to R160, R160 to R161, R161 to R162, R162 to R163, R163 to R164, R164 to R165, R165 to R166, R166 to R167, R167 to R168, R168 to R169, R169 to R170, R170 to R171, R171 to R172
